File: HDMI_RGB_Bridge/eagle/HDMI_RGB_LVDS/HDMI_RGB_LVDS.brd (EAGLE design)
At the start: 160 x 100 mm, 11 parts, among them CON1 KLDX-0202-A-LT, IC1 MBS10, IC2 TLV1117-33CDCYR

Commit message: end of workday 21.03.2014
Parts:
- added C10, C13, C14, C4, C6, C9: 100n, SchlegelAr_Master:C0603
- added C11: 1u, SchlegelAr_Master:C0603
- added C3, C5: 10u, SchlegelAr_Master:C_POL_4X4MM
- added C7, C8: 10p, SchlegelAr_Master:C0603
- added CON2: FCI-10029449-111RLF, SchlegelAr_Master:FCI-10029449-111RLF
- added CON3: XF2M-4015-1A, SchlegelAr_Master:XF2M-4015-1A
- added CON4: FCI-10033526-N3212LF, SchlegelAr_Master:FCI-10033526-N3212LF
- added CON5: MOLEX-53261-0671, SchlegelAr_Master:MOLEX-53261-0671
- added D1: BZG03C15TR3, SchlegelAr_Master:DO214A
- added IC3: TLV1117CDCYR, SchlegelAr_Master:SOT223
- added IC4: AT24C01C-SSHM-B, SchlegelAr_Master:SOIC8
- added IC5: TFP401APZP, SchlegelAr_Master:HTQFP-100
- added IC7: ATMEGA32U4-AU, SchlegelAr_Master:TQFP44
- added JP1, JP2, JP3, JP4: JUMPER3, SchlegelAr_Master:JUMPER3_THROUGHHOLE
- added JP5: (no value), SchlegelAr_Master:JUMPER2_THROUGHHOLE
- added Q1: ATS073ASM-1, SchlegelAr_Master:HC49/USSM
- added R1: 100k, SchlegelAr_Master:R0603
- added R10, R11, R12, R2, R3, R8, R9: 22R, SchlegelAr_Master:R-ARRAY-4X0603
- added R13: 4k7, SchlegelAr_Master:R0603
- added R14: 31k4, SchlegelAr_Master:R0603
- added R15, R16, R17, R4, R5, R6: 10k, SchlegelAr_Master:R0603
- added R7: 100R, SchlegelAr_Master:R0603
- added T1: IRF9530NSTRRPBF, SchlegelAr_Master:D2PAK
- C1: value 10u -> 100u
- C2: value 100u -> 10u; device SchlegelAr_Master:C_POL_6X6MM -> SchlegelAr_Master:C_POL_4X4MM
- IC1: value MBS10 -> WPMDL1300501BD; device SchlegelAr_Master:MBS -> SchlegelAr_Master:TO263-5
- IC2: value TLV1117-33CDCYR -> WPMDL1300331BD; device SchlegelAr_Master:SOT223 -> SchlegelAr_Master:TO263-5
- moved U$1 151.7 mm to (118.1, 95.2)
- moved U$2 149.8 mm to (115.6, 95.2)
- moved CON1 147.9 mm to (153.0, 5.50), turned to 90 degrees
- moved U$3 147.8 mm to (113.0, 95.2)
- moved U$15 146.7 mm to (105.4, 95.2)
- moved U$4 145.9 mm to (110.5, 95.2)
- moved U$5 144.0 mm to (108.0, 95.2)
- moved C1 128.5 mm to (142.5, 8.00), flipped to the bottom, turned to 0 degrees
- moved IC1 116.5 mm to (130.5, 7.50), turned to 0 degrees
- moved IC2 109.3 mm to (130.5, 25.5), flipped to the top, turned to 180 degrees
- moved C2 99.3 mm to (129.5, 24.0), turned to 180 degrees
Connections:
- removed net GND_EXT: CON1.1, CON1.2, IC1.AC2
- removed net VCC_EXT: CON1.3, IC1.AC1
- new net +12V: C1.+, D1.C, IC1.1, IC2.1, IC3.3, T1.3
- new net +5V: C10.2, C5.+, C9.1, CON2.18, CON4.1, CON5.5, IC1.3, IC4.8, IC7.14, IC7.2, IC7.24, IC7.34, IC7.42, IC7.44, IC7.7, R16.1, R17.2, R7.2
- new net +9V6: C3.+, CON3.2, IC3.2, IC3.4, R13.2
- new net AVR_!RESET: CON5.3, IC7.13, R16.2
- new net AVR_MISO: CON5.2
- new net AVR_MOSI: CON5.1
- new net AVR_SCK: CON5.4
- new net EDID_SCL: CON2.15, IC4.6, IC7.18
- new net EDID_SDA: CON2.16, IC4.5, IC7.19
- new net HDMI_CLK+: CON2.10, IC5.93
- new net HDMI_CLK-: CON2.12, IC5.94
- new net HDMI_DAT0+: CON2.7, IC5.90
- new net HDMI_DAT0-: CON2.9, IC5.91
- new net HDMI_DAT1+: CON2.4, IC5.85
- new net HDMI_DAT1-: CON2.6, IC5.86
- new net HDMI_DAT2+: CON2.1, IC5.80
- new net HDMI_DAT2-: CON2.3, IC5.81
- new net HDMI_OCK_INV: IC5.100, JP1.2
- new net HDMI_PIXS: IC5.4, JP2.2
- new net HDMI_ST: IC5.3, JP3.2
- new net N$1: IC5.48, R2.1M
- new net N$10: JP1.3, R6.1
- new net N$11: IC5.12, R3.2M
- new net N$12: IC5.11, R3.3M
- new net N$13: IC5.10, R3.4M
- new net N$14: IC5.17, R8.1M
- new net N$15: IC5.16, R8.2M
- new net N$16: IC5.15, R8.3M
- new net N$17: IC5.14, R8.4M
- new net N$18: CON2.19, R7.1
- new net N$19: IC5.23, R9.1M
- new net N$2: CON1.3, T1.2
- new net N$20: IC5.22, R9.2M
- new net N$21: IC5.21, R9.3M
- new net N$22: IC5.20, R9.4M
- new net N$23: IC5.27, R10.1M
- new net N$24: IC5.26, R10.2M
- new net N$25: IC5.25, R10.3M
- new net N$26: IC5.24, R10.4M
- new net N$27: IC5.33, R11.1M
- new net N$28: IC5.32, R11.2M
- new net N$29: IC5.31, R11.3M
- new net N$3: JP3.3, R4.1
- new net N$30: IC5.30, R11.4M
- new net N$31: IC5.37, R12.1M
- new net N$32: IC5.36, R12.2M
- new net N$33: IC5.35, R12.3M
- new net N$34: IC5.34, R12.4M
- new net N$35: IC3.1, R13.1, R14.1
- new net N$36: JP4.3, R15.1
- new net N$4: D1.A, R1.2, T1.1
- new net N$41: IC4.7, JP5.2, R17.1
- new net N$46: C8.2, IC7.17, Q1.1
- new net N$47: C7.2, IC7.16, Q1.2
- new net N$51: C11.2, IC7.6
- new net N$6: IC5.47, R2.2M
- new net N$7: IC5.46, R2.3M
- new net N$8: IC5.44, R2.4M
- new net N$9: IC5.13, R3.1M
- new net RGB_DE: CON3.34, R2.3P
- new net RGB_DISP: CON3.31, JP4.2
- new net RGB_HSYNC: CON3.32, R2.2P
- new net RGB_ODCK: CON3.30, R2.4P
- new net RGB_QE0: CON3.21, R3.4P
- new net RGB_QE1: CON3.22, R3.3P
- new net RGB_QE10: CON3.15, R9.2P
- new net RGB_QE11: CON3.16, R9.1P
- new net RGB_QE12: CON3.17, R10.4P
- new net RGB_QE13: CON3.18, R10.3P
- new net RGB_QE14: CON3.19, R10.2P
- new net RGB_QE15: CON3.20, R10.1P
- new net RGB_QE16: CON3.5, R11.4P
- new net RGB_QE17: CON3.6, R11.3P
- new net RGB_QE18: CON3.7, R11.2P
- new net RGB_QE19: CON3.8, R11.1P
- new net RGB_QE2: CON3.23, R3.2P
- new net RGB_QE20: CON3.9, R12.4P
- new net RGB_QE21: CON3.10, R12.3P
- new net RGB_QE22: CON3.11, R12.2P
- new net RGB_QE23: CON3.12, R12.1P
- new net RGB_QE3: CON3.24, R3.1P
- new net RGB_QE4: CON3.25, R8.4P
- new net RGB_QE5: CON3.26, R8.3P
- new net RGB_QE6: CON3.27, R8.2P
- new net RGB_QE7: CON3.28, R8.1P
- new net RGB_QE8: CON3.13, R9.4P
- new net RGB_QE9: CON3.14, R9.3P
- new net RGB_VSYNC: CON3.33, R2.1P
- new net USB_D+: CON4.3, IC7.4
- new net USB_D-: CON4.2, IC7.3
- net +3V3: now also C13.2, C14.2, C4.2, C6.2, CON3.4, IC2.3, IC5.18, IC5.29, IC5.38, IC5.43, IC5.57, IC5.6, IC5.67, IC5.78, IC5.82, IC5.84, IC5.88, IC5.95, IC5.97, IC5.99, R15.2, R4.2, R5.2, R6.2; no longer IC2.2, IC2.4
- net GND: now also C10.1, C11.1, C13.1, C14.1, C3.-, C4.1, C5.-, C6.1, C7.1, C8.1, C9.2, CON1.1, CON1.2, CON2.11, CON2.17, CON2.2, CON2.5, CON2.8, CON2.GND@1, CON2.GND@2, CON2.GND@3, CON2.GND@4, CON3.1, CON3.29, CON3.3, CON3.36, CON3.GND@1, CON3.GND@2, CON4.5, CON4.GND@1, CON4.GND@2, CON4.GND@3, CON4.GND@4, CON5.6, CON5.GND@1, CON5.GND@2, IC1.2, IC1.6, IC2.2, IC2.6, IC4.1, IC4.2, IC4.3, IC4.4, IC5.1, IC5.19, IC5.28, IC5.39, IC5.45, IC5.5, IC5.58, IC5.68, IC5.7, IC5.76, IC5.79, IC5.83, IC5.87, IC5.89, IC5.92, IC5.98, IC7.15, IC7.23, IC7.35, IC7.43, IC7.5, JP1.1, JP2.1, JP3.1, JP4.1, JP5.1, R1.1, R14.2; no longer IC1.-, IC2.1
- net N$5: now also JP2.3, R5.1; no longer C1.+, IC1.+, IC2.3

Commit message: end of workday 22.03.2014
Parts:
- added C12: 100n, SchlegelAr_Master:C0603
- added C15, C17, C19, C21, C22: 0.01u, SchlegelAr_Master:C0603
- added C16, C18, C20: 0.1u, SchlegelAr_Master:C0603
- added CON6: FI-X30SSLA-HF, SchlegelAr_Master:FI-X30SSLA-HF
- added IC6: ATMEGA48A-AU, SchlegelAr_Master:TQFP32
- added IC8: SN75LVDS83BDGGR, SchlegelAr_Master:TSSOP-56
- added JP6: (no value), SchlegelAr_Master:JUMPER2_THROUGHHOLE
- added JP7, JP8: JUMPER3, SchlegelAr_Master:JUMPER3_THROUGHHOLE
- added R18: 10k, SchlegelAr_Master:R0603
- C11: value 1u -> 100n
- IC7: value ATMEGA32U4-AU -> FT232RL; device SchlegelAr_Master:TQFP44 -> SchlegelAr_Master:SSOP28
- JP1, JP2, JP3: value JUMPER3 -> (none)
- moved C1 59.0 mm to (83.5, 8.00)
- moved C2 59.0 mm to (70.5, 24.0)
- moved C3 59.0 mm to (77.0, 26.5)
- moved C5 59.0 mm to (71.0, 8.00)
- moved CON1 59.0 mm to (94.0, 5.50)
- moved D1 59.0 mm to (83.5, 21.0)
- moved IC1 59.0 mm to (71.5, 7.50)
- moved IC2 59.0 mm to (71.5, 25.5)
- moved IC3 59.0 mm to (82.0, 29.5)
- moved R1 59.0 mm to (87.5, 17.5)
- moved R13 59.0 mm to (81.5, 24.0)
- moved R14 59.0 mm to (78.5, 23.5)
- moved T1 59.0 mm to (83.0, 8.00)
- moved IC7 14.7 mm to (7.00, 7.00), flipped to the bottom, turned to 180 degrees
- moved JP5 14.3 mm to (7.00, 16.0), turned to 180 degrees
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Connections:
- net N$41 renamed EDID_WRITEPROTECT
- removed net N$46: C8.2, IC7.17, Q1.1
- removed net N$47: C7.2, IC7.16, Q1.2
- removed net N$51: C11.2, IC7.6
- removed net RGB_QE0: CON3.21, R3.4P
- removed net RGB_QE1: CON3.22, R3.3P
- removed net RGB_QE10: CON3.15, R9.2P
- removed net RGB_QE11: CON3.16, R9.1P
- removed net RGB_QE12: CON3.17, R10.4P
- removed net RGB_QE13: CON3.18, R10.3P
- removed net RGB_QE14: CON3.19, R10.2P
- removed net RGB_QE15: CON3.20, R10.1P
- removed net RGB_QE16: CON3.5, R11.4P
- removed net RGB_QE17: CON3.6, R11.3P
- removed net RGB_QE18: CON3.7, R11.2P
- removed net RGB_QE19: CON3.8, R11.1P
- removed net RGB_QE2: CON3.23, R3.2P
- removed net RGB_QE20: CON3.9, R12.4P
- removed net RGB_QE21: CON3.10, R12.3P
- removed net RGB_QE22: CON3.11, R12.2P
- removed net RGB_QE23: CON3.12, R12.1P
- removed net RGB_QE3: CON3.24, R3.1P
- removed net RGB_QE4: CON3.25, R8.4P
- removed net RGB_QE5: CON3.26, R8.3P
- removed net RGB_QE6: CON3.27, R8.2P
- removed net RGB_QE7: CON3.28, R8.1P
- removed net RGB_QE8: CON3.13, R9.4P
- removed net RGB_QE9: CON3.14, R9.3P
- new net AREF: IC6.20
- new net AVR_PWM: IC6.13, JP8.2
- new net AVR_XTAL1: C7.2, IC6.7, Q1.2
- new net AVR_XTAL2: C8.2, IC6.8, Q1.1
- new net FTDI_3V3OUT: C11.1, IC7.17, IC7.4
- new net FTDI_RXD: IC6.31, IC7.5
- new net FTDI_TXD: IC6.30, IC7.1
- new net LVDS_0+: CON6.8, IC8.47
- new net LVDS_0-: CON6.7, IC8.48
- new net LVDS_1+: CON6.11, IC8.45
- new net LVDS_1-: CON6.10, IC8.46
- new net LVDS_2+: CON6.14, IC8.41
- new net LVDS_2-: CON6.13, IC8.42
- new net LVDS_3+: CON6.20, IC8.37
- new net LVDS_3-: CON6.19, IC8.38
- new net LVDS_CLK+: CON6.17, IC8.39
- new net LVDS_CLK-: CON6.16, IC8.40
- new net LVDS_PWM: CON6.24, JP8.3
- new net LVDS_REVSCAN: CON6.5, JP7.2
- new net N$37: CON3.2, JP6.2
- new net N$38: JP7.3, R18.1
- new net N$40: CON6.25
- new net RGB_EVEN_B0: CON3.21, IC8.15, R3.4P
- new net RGB_EVEN_B1: CON3.22, IC8.19, R3.3P
- new net RGB_EVEN_B2: CON3.23, IC8.20, R3.2P
- new net RGB_EVEN_B3: CON3.24, IC8.22, R3.1P
- new net RGB_EVEN_B4: CON3.25, IC8.23, R8.4P
- new net RGB_EVEN_B5: CON3.26, IC8.24, R8.3P
- new net RGB_EVEN_B6: CON3.27, IC8.16, R8.2P
- new net RGB_EVEN_B7: CON3.28, IC8.18, R8.1P
- new net RGB_EVEN_G0: CON3.13, IC8.4, R9.4P
- new net RGB_EVEN_G1: CON3.14, IC8.6, R9.3P
- new net RGB_EVEN_G2: CON3.15, IC8.7, R9.2P
- new net RGB_EVEN_G3: CON3.16, IC8.11, R9.1P
- new net RGB_EVEN_G4: CON3.17, IC8.12, R10.4P
- new net RGB_EVEN_G5: CON3.18, IC8.14, R10.3P
- new net RGB_EVEN_G6: CON3.19, IC8.8, R10.2P
- new net RGB_EVEN_G7: CON3.20, IC8.10, R10.1P
- new net RGB_EVEN_R0: CON3.5, IC8.51, R11.4P
- new net RGB_EVEN_R1: CON3.6, IC8.52, R11.3P
- new net RGB_EVEN_R2: CON3.7, IC8.54, R11.2P
- new net RGB_EVEN_R3: CON3.8, IC8.55, R11.1P
- new net RGB_EVEN_R4: CON3.9, IC8.56, R12.4P
- new net RGB_EVEN_R5: CON3.10, IC8.3, R12.3P
- new net RGB_EVEN_R6: CON3.11, IC8.50, R12.2P
- new net RGB_EVEN_R7: CON3.12, IC8.2, R12.1P
- new net RGB_PWM: JP8.1
- net +12V: now also CON6.28, CON6.29, CON6.30
- net +3V3: now also C15.2, C16.2, C17.2, C18.2, C19.2, C20.2, C21.2, C22.2, CON6.1, CON6.2, IC8.1, IC8.26, IC8.34, IC8.44, IC8.9, R18.2
- net +5V: now also C12.1, IC6.18, IC6.4, IC6.6, IC7.19, IC7.20; no longer IC7.14, IC7.2, IC7.24, IC7.34, IC7.42, IC7.44, IC7.7
- net +9V6: now also JP6.1; no longer CON3.2
- net AVR_!RESET: now also IC6.29; no longer IC7.13
- net AVR_MISO: now also IC6.16
- net AVR_MOSI: now also IC6.15
- net AVR_SCK: now also IC6.17
- net EDID_SCL: now also IC6.28; no longer IC7.18
- net EDID_SDA: now also IC6.27; no longer IC7.19
- net GND: now also C11.2, C12.2, C15.1, C16.1, C17.1, C18.1, C19.1, C20.1, C21.1, C22.1, CON6.12, CON6.15, CON6.18, CON6.21, CON6.26, CON6.3, CON6.4, CON6.6, CON6.9, CON6.GND@1, CON6.GND@2, CON6.GND@3, CON6.GND@4, IC6.21, IC6.3, IC6.5, IC7.18, IC7.21, IC7.25, IC7.26, IC7.7, IC8.13, IC8.21, IC8.25, IC8.29, IC8.33, IC8.35, IC8.36, IC8.43, IC8.49, IC8.5, IC8.53, JP7.1; no longer C11.1, IC7.15, IC7.23, IC7.35, IC7.43, IC7.5
- net RGB_DE: now also IC8.30
- net RGB_HSYNC: now also IC8.27
- net RGB_ODCK: now also IC8.31
- net RGB_VSYNC: now also IC8.28
- net USB_D+: now also IC7.16; no longer IC7.4
- net USB_D-: now also IC7.15; no longer IC7.3
Other:
- board size 160 x 100 mm -> 99.8 x 100 mm

Commit message: commit mid 24.03.2014
Parts:
- added C23, C24: 100n, SchlegelAr_Master:C0402
- added R19: 10k, SchlegelAr_Master:35WR5KLFTR
- added R20, R21: 140R, SchlegelAr_Master:R2512
- added SP1, SP10, SP11, SP12, SP13, SP14, SP15, SP16, SP17, SP18, SP2, SP3, SP4, SP5, SP9, U$95, U$96, U$97: SP2, SchlegelAr_Master:SP2
- added T2: IRLML2502TRPBF, SchlegelAr_Master:SOT23
- C10, C11, C12, C13, C14, C15, C16, C17, C18, C19, C20, C21, C22, C4, C6, C7, C8, C9: device SchlegelAr_Master:C0603 -> SchlegelAr_Master:C0402
- JP1, JP2, JP3: value (none) -> JUMPER2; device SchlegelAr_Master:JUMPER3_THROUGHHOLE -> SchlegelAr_Master:JUMPER2_THROUGHHOLE
- JP6: value (none) -> JUMPER3; device SchlegelAr_Master:JUMPER2_THROUGHHOLE -> SchlegelAr_Master:JUMPER3_THROUGHHOLE
- JP7, JP8: value JUMPER3 -> (none); device SchlegelAr_Master:JUMPER3_THROUGHHOLE -> SchlegelAr_Master:JUMPER2_THROUGHHOLE
- R1, R13, R14, R15, R16, R17, R18, R4, R5, R6, R7: device SchlegelAr_Master:R0603 -> SchlegelAr_Master:R0402
- moved U$2 149.8 mm to (0.00, 0.00)
- moved U$3 147.8 mm to (0.00, 0.00)
- moved U$4 145.9 mm to (0.00, 0.00)
- moved U$5 144.0 mm to (0.00, 0.00)
- moved U$1 142.5 mm to (12.7, -0.62)
- moved U$15 142.1 mm to (0.00, 0.00)
- moved JP7 66.3 mm to (14.6, 17.6), turned to 90 degrees
- moved CON6 62.1 mm to (5.00, 38.4), flipped to the bottom, turned to 270 degrees
- moved R18 59.9 mm to (11.4, 17.6), turned to 270 degrees
- moved R4 45.5 mm to (11.4, 21.4)
- moved C19 43.0 mm to (18.5, 37.5), turned to 180 degrees
- moved C17 42.9 mm to (21.0, 43.0)
- moved C20 42.5 mm to (18.5, 36.0), turned to 180 degrees
- moved C18 41.6 mm to (18.4, 40.9), turned to 180 degrees
- moved C15 41.4 mm to (18.4, 42.6), turned to 180 degrees
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Connections:
- net EDID_WRITEPROTECT renamed EDID_WP
- removed net AREF: IC6.20
- removed net HDMI_ST: IC5.3, JP3.2
- removed net N$10: JP1.3, R6.1
- removed net N$3: JP3.3, R4.1
- removed net N$36: JP4.3, R15.1
- removed net N$38: JP7.3, R18.1
- removed net N$40: CON6.25
- removed net N$5: JP2.3, R5.1
- new net AVR_PWM_ADC: IC6.23, R19.2
- new net LVDS_LED_EN: CON6.25, JP8.2, R4.1
- new net N$39: C22.2, IC8.1, SP15.P$1
- new net N$41: C21.2, IC8.26, SP16.P$1
- new net N$42: C15.2, C18.2, IC8.44, SP17.P$1
- new net N$43: C19.2, C20.2, IC8.34, SP18.P$1
- new net N$44: C12.1, IC7.20, SP9.P$1
- new net N$45: C24.1, IC6.18, SP13.P$2
- new net N$46: C9.1, IC6.4, SP11.P$2
- new net N$47: C23.1, IC6.6, SP12.P$2
- new net N$48: C16.2, C17.2, IC8.9, SP14.P$1
- new net N$49: C10.2, IC4.8, SP10.P$2
- new net N$50: C6.2, IC5.18, IC5.29, IC5.43, IC5.57, IC5.78, SP4.P$1
- new net N$51: C2.+, U$96.P$1
- new net N$52: C4.2, IC5.82, IC5.84, IC5.88, IC5.95, SP5.P$1
- new net N$53: C13.2, IC5.97, SP2.P$1
- new net N$54: C14.2, IC5.38, IC5.6, IC5.67, SP3.P$1
- new net N$55: C3.+, U$97.P$1
- new net N$56: C5.+, U$95.P$1
- new net N$57: R20.1, R21.1, T2.3
- new net N$59: C1.+, D1.C, IC1.1, IC2.1, IC3.3, SP1.P$1, T1.3
- new net RGB_PWM_EN: JP4.2, T2.1
- net +12V: now also SP1.P$2; no longer C1.+, D1.C, IC1.1, IC2.1, IC3.3, T1.3
- net +3V3: now also JP4.1, SP14.P$2, SP15.P$2, SP16.P$2, SP17.P$2, SP18.P$2, SP2.P$2, SP3.P$2, SP4.P$2, SP5.P$2, U$96.P$2; no longer C13.2, C14.2, C15.2, C16.2, C17.2, C18.2, C19.2, C2.+, C20.2, C21.2, C22.2, C4.2, C6.2, IC5.18, IC5.29, IC5.38, IC5.43, IC5.57, IC5.6, IC5.67, IC5.78, IC5.82, IC5.84, IC5.88, IC5.95, IC5.97, IC8.1, IC8.26, IC8.34, IC8.44, IC8.9
- net +5V: now also IC6.20, IC7.4, R19.1, SP10.P$1, SP11.P$1, SP12.P$1, SP13.P$1, SP9.P$2, U$95.P$2; no longer C10.2, C12.1, C5.+, C9.1, IC4.8, IC6.18, IC6.4, IC6.6, IC7.20
- net +9V6: now also R20.2, R21.2, U$97.P$2; no longer C3.+, JP6.1
- net AVR_PWM: now also JP6.2; no longer JP8.2
- net FTDI_3V3OUT: no longer IC7.4
- net GND: now also C23.2, C24.2, IC5.3, JP8.1, R19.3; no longer JP4.1
- net HDMI_OCK_INV: now also R6.1
- net HDMI_PIXS: now also R5.1
- net LVDS_PWM: now also JP6.3; no longer JP8.3
- net LVDS_REVSCAN: now also R18.1
- net N$37: now also T2.2; no longer JP6.2
- net RGB_DISP: now also JP3.2, R15.1; no longer JP4.2
- net RGB_PWM: now also JP4.3, JP6.1; no longer JP8.1
Routing:
- added copper zone on layer 2, net GND
Other:
- board size 99.8 x 100 mm -> 90 x 60 mm

Commit message: end of workday 24.03.2014
Parts:
- added R22, R23: 0R, SchlegelAr_Master:R0402
- moved C3 4.95 mm to (65.5, 44.5), turned to 180 degrees
- moved U$97 2.30 mm to (67.2, 48.1)
- moved SP12 1.94 mm to (22.3, 11.1), turned to 180 degrees
- moved SP11 1.46 mm to (25.5, 8.75)
- moved SP10 1.31 mm to (16.9, 8.06), turned to 90 degrees
- moved SP1 1.27 mm to (67.9, 27.6)
- moved JP5 0.40 mm to (19.5, 2.25)
- moved SP9 0.25 mm to (6.62, 10.9), turned to 180 degrees
Connections:
- new net N$10: IC7.16, R23.2
- new net N$5: IC7.15, R22.2
- net USB_D+: now also R23.1; no longer IC7.16
- net USB_D-: now also R22.1; no longer IC7.15
Routing:
- net GND: track 0.00 -> 74.3 mm, vias 0 -> 26
- net N$59: track 0.00 -> 42.5 mm, vias 0 -> 3
- net AVR_!RESET: track 0.00 -> 23.7 mm
- net +5V: track 0.00 -> 20.4 mm, vias 0 -> 11
- net FTDI_RXD: track 0.00 -> 19.3 mm, vias 0 -> 1
- net AVR_MOSI: track 0.00 -> 16.3 mm
- net +9V6: track 0.00 -> 15.1 mm
- net N$2: track 0.00 -> 14.9 mm
- net HDMI_PIXS: track 0.00 -> 13.6 mm
- net AVR_MISO: track 0.00 -> 13.4 mm
- net FTDI_TXD: track 0.00 -> 12.8 mm, vias 0 -> 1
- net EDID_SCL: track 0.00 -> 12.4 mm, vias 0 -> 1
- net AVR_SCK: track 0.00 -> 11.4 mm
- net EDID_SDA: track 0.00 -> 10.8 mm, vias 0 -> 1
- net AVR_XTAL2: track 0.00 -> 10.6 mm
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- added copper zone on layer 15, net +5V
