File: HDMI_RGB_Bridge/eagle/HDMI_RGB_LVDS/HDMI_RGB_LVDS.sch (EAGLE design)
At the start: 11 parts, among them CON1 KLDX-0202-A-LT, IC1 MBS10, IC2 TLV1117-33CDCYR

Commit message: end of workday 20.03.2014
Other:
- note added: "AVR ISP"
- note added: "AVR ISP Connector Molex 53261-0671"
- note added: "Atmel ATmega48"
- note added: "Blockschaltbild"
- note added: "Edid data"
- note added: "Erstellung des Projekts, S2: Blockschaltbild, S3: Spannungsversorgung +3.3V hinzugefuegt"
- note added: "HDMI"
- note added: "HDMI Connector FCI 10029449-111RLF"
- note added: "HDMI RGB Bridge TI TFP401A"
- note added: "I2C"
- note added: "I2C EEPROM Atmel AT2401C"
- note added: "LVDS"
- note added: "LVDS Connector JAE FI-X30SSLA-HF"
- note added: "LVDS Display LG LB070WV8-SL01"
- note added: "Mini USB Connector FCI 10033526-N3212LF"
- note added: "RGB Bus"
- note added: "RGB Connector OMRON XF2M-4015-1A"
- note added: "RGB Display"
- note added: "RGB LVDS Bridge TI SN75LVDS83B"
- note added: "RS232-USB-Bridge FTDI FT232RL"
- note added: "UART"
- note added: "USB"
- note removed: "Erstellung des Projekts, S3: Spannungsversorgung +3.3V hinzugefuegt"
Changed lines of the file:
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@@
 <sheet>
 <plain>
-<text x="35.56" y="210.82" size="2.54" layer="94">Erstellung des Projekts, S3: Spannungsversorgung +3.3V hinzugefuegt</text>
+<text x="35.56" y="210.82" size="2.54" layer="94">Erstellung des Projekts, S2: Blockschaltbild, S3: Spannungsversorgung +3.3V hinzugefuegt</text>
 <text x="10.16" y="246.38" size="5.08" layer="94">HDMI_RGB_LVDS</text>
 <text x="83.82" y="246.38" size="5.08" layer="94">Masterarbeit Armin Schlegel SS14</text>
@@
 <sheet>
 <plain>
+<wire x1="20.32" y1="231.14" x2="20.32" y2="210.82" width="0.6096" layer="94"/>
+<wire x1="20.32" y1="210.82" x2="68.58" y2="210.82" width="0.6096" layer="94"/>
+<wire x1="68.58" y1="210.82" x2="68.58" y2="231.14" width="0.6096" layer="94"/>
+<wire x1="68.58" y1="231.14" x2="20.32" y2="231.14" width="0.6096" layer="94"/>
+<text x="22.86" y="215.9" size="2.54" layer="94">HDMI Connector
+FCI 10029449-111RLF</text>
+<wire x1="276.86" y1="231.14" x2="276.86" y2="210.82" width="0.6096" layer="94"/>
+<wire x1="276.86" y1="210.82" x2="325.12" y2="210.82" width="0.6096" layer="94"/>
+<wire x1="325.12" y1="210.82" x2="325.12" y2="231.14" width="0.6096" layer="94"/>
+<wire x1="325.12" y1="231.14" x2="276.86" y2="231.14" width="0.6096" layer="94"/>
+<text x="279.4" y="215.9" size="2.54" layer="94">LVDS Display
+LG LB070WV8-SL01</text>
+<wire x1="276.86" y1="203.2" x2="276.86" y2="182.88" width="0.6096" layer="94"/>
+<wire x1="276.86" y1="182.88" x2="325.12" y2="182.88" width="0.6096" layer="94"/>
+<wire x1="325.12" y1="182.88" x2="325.12" y2="203.2" width="0.6096" layer="94"/>
+<wire x1="325.12" y1="203.2" x2="276.86" y2="203.2" width="0.6096" layer="94"/>
+<text x="281.94" y="193.04" size="2.54" layer="94">RGB Display</text>
+<wire x1="127" y1="231.14" x2="127" y2="210.82" width="0.6096" layer="94"/>
+<wire x1="127" y1="210.82" x2="86.36" y2="210.82" width="0.6096" layer="94"/>
+<wire x1="86.36" y1="210.82" x2="86.36" y2="231.14" width="0.6096" layer="94"/>
+<wire x1="86.36" y1="231.14" x2="127" y2="231.14" width="0.6096" layer="94"/>
+<wire x1="195.58" y1="231.14" x2="195.58" y2="210.82" width="0.6096" layer="94"/>
+<wire x1="195.58" y1="210.82" x2="154.94" y2="210.82" width="0.6096" layer="94"/>
+<wire x1="154.94" y1="210.82" x2="154.94" y2="231.14" width="0.6096" layer="94"/>
+<wire x1="154.94" y1="231.14" x2="195.58" y2="231.14" width="0.6096" layer="94"/>
+<wire x1="60.96" y1="190.5" x2="60.96" y2="167.64" width="0.6096" layer="94"/>
+<wire x1="60.96" y1="167.64" x2="20.32" y2="167.64" width="0.6096" layer="94"/>
+<wire x1="20.32" y1="167.64" x2="20.32" y2="190.5" width="0.6096" layer="94"/>
+<wire x1="20.32" y1="190.5" x2="60.96" y2="190.5" width="0.6096" layer="94"/>
+<wire x1="60.96" y1="157.48" x2="60.96" y2="134.62" width="0.6096" layer="94"/>
+<wire x1="60.96" y1="134.62" x2="20.32" y2="134.62" width="0.6096" layer="94"/>
+<wire x1="20.32" y1="134.62" x2="20.32" y2="157.48" width="0.6096" layer="94"/>
+<wire x1="20.32" y1="157.48" x2="60.96" y2="157.48" width="0.6096" layer="94"/>
+<wire x1="60.96" y1="124.46" x2="60.96" y2="101.6" width="0.6096" layer="94"/>
+<wire x1="60.96" y1="101.6" x2="20.32" y2="101.6" width="0.6096" layer="94"/>
+<wire x1="20.32" y1="101.6" x2="20.32" y2="124.46" width="0.6096" layer="94"/>
+<wire x1="20.32" y1="124.46" x2="60.96" y2="124.46" width="0.6096" layer="94"/>
+<wire x1="20.32" y1="88.9" x2="20.32" y2="66.04" width="0.6096" layer="94"/>
+<wire x1="20.32" y1="66.04" x2="71.12" y2="66.04" width="0.6096" layer="94"/>
+<wire x1="71.12" y1="66.04" x2="71.12" y2="88.9" width="0.6096" layer="94"/>
+<wire x1="71.12" y1="88.9" x2="20.32" y2="88.9" width="0.6096" layer="94"/>
+<text x="22.86" y="71.12" size="2.54" layer="94">Mini USB
+Connector
+FCI 10033526-N3212LF</text>
+<wire x1="78.74" y1="88.9" x2="78.74" y2="66.04" width="0.6096" layer="94"/>
+<wire x1="78.74" y1="66.04" x2="137.16" y2="66.04" width="0.6096" layer="94"/>
+<wire x1="137.16" y1="66.04" x2="137.16" y2="88.9" width="0.6096" layer="94"/>
+<wire x1="137.16" y1="88.9" x2="78.74" y2="88.9" width="0.6096" layer="94"/>
+<text x="81.28" y="71.12" size="2.54" layer="94">AVR ISP
+Connector
+Molex 53261-0671</text>
+<wire x1="215.9" y1="231.14" x2="215.9" y2="210.82" width="0.6096" layer="94"/>
+<wire x1="215.9" y1="210.82" x2="261.62" y2="210.82" width="0.6096" layer="94"/>
+<wire x1="261.62" y1="210.82" x2="261.62" y2="231.14" width="0.6096" layer="94"/>
+<wire x1="261.62" y1="231.14" x2="215.9" y2="231.14" width="0.6096" layer="94"/>
+<text x="218.44" y="215.9" size="2.54" layer="94">LVDS Connector
+JAE FI-X30SSLA-HF</text>
+<wire x1="215.9" y1="203.2" x2="215.9" y2="182.88" width="0.6096" layer="94"/>
+<wire x1="215.9" y1="182.88" x2="261.62" y2="182.88" width="0.6096" layer="94"/>
+<wire x1="261.62" y1="182.88" x2="261.62" y2="203.2" width="0.6096" layer="94"/>
+<wire x1="261.62" y1="203.2" x2="215.9" y2="203.2" width="0.6096" layer="94"/>
+<text x="218.44" y="187.96" size="2.54" layer="94">RGB Connector
+OMRON XF2M-4015-1A</text>
+<text x="88.9" y="215.9" size="2.54" layer="94">HDMI RGB Bridge
+TI TFP401A</text>
+<text x="157.48" y="215.9" size="2.54" layer="94">RGB LVDS Bridge
+TI SN75LVDS83B</text>
+<text x="22.86" y="175.26" size="2.54" layer="94">I2C EEPROM
+Atmel AT2401C</text>
+<text x="22.86" y="144.78" size="2.54" layer="94">Atmel ATmega48</text>
+<text x="22.86" y="106.68" size="2.54" layer="94">RS232-USB-Bridge
+FTDI FT232RL</text>
+<text x="40.64" y="195.58" size="2.54" layer="97">Edid data</text>
+<text x="134.62" y="223.52" size="2.54" layer="97">RGB Bus</text>
+<text x="200.66" y="223.52" size="2.54" layer="97">LVDS</text>
+<text x="40.64" y="203.2" size="2.54" layer="97">I2C</text>
+<text x="40.64" y="162.56" size="2.54" layer="97">I2C</text>
+<text x="40.64" y="129.54" size="2.54" layer="97">UART</text>
+<text x="40.64" y="93.98" size="2.54" layer="97">USB</text>
+<text x="68.58" y="147.32" size="2.54" layer="97">AVR ISP</text>
+<text x="73.66" y="223.52" size="2.54" layer="97">HDMI</text>
+<text x="20.32" y="236.22" size="6.4516" layer="97">Blockschaltbild</text>
 </plain>
 <instances>
@@
 </instances>
 <busses>
+<bus name="B$1">
+<segment>
+<wire x1="68.58" y1="220.98" x2="86.36" y2="220.98" width="1.6764" layer="92"/>
+</segment>
+</bus>
+<bus name="B$2">
+<segment>
+<wire x1="127" y1="220.98" x2="154.94" y2="220.98" width="1.6764" layer="92"/>
+</segment>
+</bus>
+<bus name="B$3">
+<segment>
+<wire x1="195.58" y1="220.98" x2="215.9" y2="220.98" width="1.6764" layer="92"/>
+</segment>
+</bus>
+<bus name="B$4">
+<segment>
+<wire x1="261.62" y1="220.98" x2="276.86" y2="220.98" width="1.6764" layer="92"/>
+</segment>
+</bus>
+<bus name="B$5">
+<segment>
+<wire x1="261.62" y1="193.04" x2="276.86" y2="193.04" width="1.6764" layer="92"/>
+</segment>
+</bus>
+<bus name="B$6">
+<segment>
+<wire x1="215.9" y1="193.04" x2="142.24" y2="193.04" width="1.6764" layer="92"/>
+<wire x1="142.24" y1="193.04" x2="142.24" y2="220.98" width="1.6764" layer="92"/>
+</segment>
+</bus>
+<bus name="B$7">
+<segment>
+<wire x1="38.1" y1="190.5" x2="38.1" y2="210.82" width="1.6764" layer="92"/>
+</segment>
+</bus>
+<bus name="B$8">
+<segment>
+<wire x1="38.1" y1="157.48" x2="38.1" y2="167.64" width="1.6764" layer="92"/>
+</segment>
+</bus>
+<bus name="B$9">
+<segment>
+<wire x1="38.1" y1="124.46" x2="38.1" y2="134.62" width="1.6764" layer="92"/>
+</segment>
+</bus>
+<bus name="B$10">
+<segment>
+<wire x1="38.1" y1="88.9" x2="38.1" y2="101.6" width="1.6764" layer="92"/>
+</segment>
+</bus>
+<bus name="B$11">
+<segment>
+<wire x1="106.68" y1="88.9" x2="106.68" y2="144.78" width="1.6764" layer="92"/>
+<wire x1="106.68" y1="144.78" x2="60.96" y2="144.78" width="1.6764" layer="92"/>
+</segment>
+</bus>
 </busses>
 <nets>
@@
 </schematic>
 </drawing>
+<compatibility>
+<note version="6.3" minversion="6.2.2" severity="warning">
+Since Version 6.2.2 text objects can contain more than one line,
+which will not be processed correctly with this version.
+</note>
+</compatibility>
 </eagle>

Commit message: end of workday 21.03.2014
Parts:
- added C10, C13, C14, C4, C6, C9: 100n, SchlegelAr_Master:C_SMD0603
- added C11: 1u, SchlegelAr_Master:C_SMD0603
- added C3, C5: 10u, SchlegelAr_Master:C_POL4X4MM
- added C7, C8: 10p, SchlegelAr_Master:C_SMD0603
- added CON2: FCI-10029449-111RLF, SchlegelAr_Master:FCI-10029449-111RLF
- added CON3: XF2M-4015-1A, SchlegelAr_Master:XF2M-4015-1A
- added CON4: FCI-10033526-N3212LF, SchlegelAr_Master:FCI-10033526-N3212LF
- added CON5: MOLEX-53261-0671, SchlegelAr_Master:MOLEX-53261-0671
- added D1: BZG03C15TR3, SchlegelAr_Master:BZG03C15TR3
- added IC3: TLV1117CDCYR, SchlegelAr_Master:TLV1117CDCYR
- added IC4: AT24C01C-SSHM-B, SchlegelAr_Master:AT24C01C-SSHM-B
- added IC5: TFP401APZP, SchlegelAr_Master:TFP401APZP
- added IC7: ATMEGA32U4-AU, SchlegelAr_Master:ATMEGA32U4-AU
- added JP1, JP2, JP3, JP4: JUMPER3, SchlegelAr_Master:JUMPER3
- added JP5: JUMPER2THROUGHHOLE_2.54MM, SchlegelAr_Master:JUMPER2THROUGHHOLE_2.54MM
- added Q1: ATS073ASM-1, SchlegelAr_Master:ATS073ASM-1
- added R1: 100k, SchlegelAr_Master:R0603
- added R10, R11, R12, R2, R3, R8, R9: 22R, SchlegelAr_Master:CTR-742C083220JP-4X22R-4X0603
- added R13: 4k7, SchlegelAr_Master:R0603
- added R14: 31k4, SchlegelAr_Master:R0603
- added R15, R16, R17, R4, R5, R6: 10k, SchlegelAr_Master:R0603
- added R7: 100R, SchlegelAr_Master:R0603
- added T1: IRF9530NSTRRPBF, SchlegelAr_Master:IRF9530NSTRRPBF
- C1: value 10u -> 100u
- C2: value 100u -> 10u; device SchlegelAr_Master:C_POL6X6MM -> SchlegelAr_Master:C_POL4X4MM
- IC1: value MBS10 -> WPMDL1300501BD; device SchlegelAr_Master:MBS10 -> SchlegelAr_Master:WPMDL1300501BD
- IC2: value TLV1117-33CDCYR -> WPMDL1300331BD; device SchlegelAr_Master:TLV1117-33CDCYR -> SchlegelAr_Master:WPMDL1300331BD
Connections:
- removed net GND_EXT: CON1.2, CON1.3, IC1.AC2
- removed net VCC_EXT: CON1.1, IC1.AC1
- new net +12V: C1.P$1, D1.C, IC1.VIN, IC2.VIN, IC3.IN, T1.S
- new net +5V: C10.P$2, C5.P$1, C9.P$1, CON2.+5V, CON4.VBUS, CON5.VCC, IC1.VOUT, IC4.VCC, IC7.AREF, IC7.AVCC@1, IC7.AVCC@2, IC7.UVCC, IC7.VBUS, IC7.VCC@1, IC7.VCC@2, R16.P$1, R17.P$2, R7.P$2
- new net +9V6: C3.P$1, CON3.LED-A, IC3.OUT, IC3.OUT1, R13.P$2
- new net AVR_!RESET: CON5.RESET, IC7.!RESET, R16.P$2
- new net AVR_MISO: CON5.MISO
- new net AVR_MOSI: CON5.MOSI
- new net AVR_SCK: CON5.SCK
- new net EDID_SCL: CON2.SCL, IC4.SCL, IC7.PD0(INT0/OC0B/SCL)
- new net EDID_SDA: CON2.SDA, IC4.SDA, IC7.PD1(INT1/SDA)
- new net HDMI_CLK+: CON2.CLK+, IC5.RXC+
- new net HDMI_CLK-: CON2.CLK-, IC5.RXC-
- new net HDMI_DAT0+: CON2.DATA0+, IC5.RX0+
- new net HDMI_DAT0-: CON2.DATA0-, IC5.RX0-
- new net HDMI_DAT1+: CON2.DATA1+, IC5.RX1+
- new net HDMI_DAT1-: CON2.DATA1-, IC5.RX1-
- new net HDMI_DAT2+: CON2.DATA2+, IC5.RX2+
- new net HDMI_DAT2-: CON2.DATA2-, IC5.RX2-
- new net HDMI_OCK_INV: IC5.OCK_INV, JP1.2
- new net HDMI_PIXS: IC5.PIXS, JP2.2
- new net HDMI_ST: IC5.ST, JP3.2
- new net N$1: IC5.HSYNC, R2.1M
- new net N$10: JP1.3, R6.P$1
- new net N$11: IC5.QE2, R3.2M
- new net N$12: IC5.QE1, R3.3M
- new net N$13: IC5.QE0, R3.4M
- new net N$14: IC5.QE7, R8.1M
- new net N$15: IC5.QE6, R8.2M
- new net N$16: IC5.QE5, R8.3M
- new net N$17: IC5.QE4, R8.4M
- new net N$18: CON2.DETECT, R7.P$1
- new net N$19: IC5.QE11, R9.1M
- new net N$2: CON1.1, T1.D
- new net N$20: IC5.QE10, R9.2M
- new net N$21: IC5.QE9, R9.3M
- new net N$22: IC5.QE8, R9.4M
- new net N$23: IC5.QE15, R10.1M
- new net N$24: IC5.QE14, R10.2M
- new net N$25: IC5.QE13, R10.3M
- new net N$26: IC5.QE12, R10.4M
- new net N$27: IC5.QE19, R11.1M
- new net N$28: IC5.QE18, R11.2M
- new net N$29: IC5.QE17, R11.3M
- new net N$3: JP3.3, R4.P$1
- new net N$30: IC5.QE16, R11.4M
- new net N$31: IC5.QE23, R12.1M
- new net N$32: IC5.QE22, R12.2M
- new net N$33: IC5.QE21, R12.3M
- new net N$34: IC5.QE20, R12.4M
- new net N$35: IC3.GND, R13.P$1, R14.P$1
- new net N$36: JP4.3, R15.P$1
- new net N$4: D1.A, R1.P$2, T1.G
- new net N$41: IC4.WP, JP5.2, R17.P$1
- new net N$46: C8.P$2, IC7.XTAL1, Q1.1
- new net N$47: C7.P$2, IC7.XTAL2, Q1.2
- new net N$51: C11.P$2, IC7.UCAP
- new net N$6: IC5.VSYNC, R2.2M
- new net N$7: IC5.DE, R2.3M
- new net N$8: IC5.ODCK, R2.4M
- new net N$9: IC5.QE3, R3.1M
- new net RGB_DE: CON3.DEN, R2.3P
- new net RGB_DISP: CON3.DISP, JP4.2
- new net RGB_HSYNC: CON3.HSYNC, R2.2P
- new net RGB_ODCK: CON3.CLK, R2.4P
- new net RGB_QE0: CON3.B0, R3.4P
- new net RGB_QE1: CON3.B1, R3.3P
- new net RGB_QE10: CON3.G2, R9.2P
- new net RGB_QE11: CON3.G3, R9.1P
- new net RGB_QE12: CON3.G4, R10.4P
- new net RGB_QE13: CON3.G5, R10.3P
- new net RGB_QE14: CON3.G6, R10.2P
- new net RGB_QE15: CON3.G7, R10.1P
- new net RGB_QE16: CON3.R0, R11.4P
- new net RGB_QE17: CON3.R1, R11.3P
- new net RGB_QE18: CON3.R2, R11.2P
- new net RGB_QE19: CON3.R3, R11.1P
- new net RGB_QE2: CON3.B2, R3.2P
- new net RGB_QE20: CON3.R4, R12.4P
- new net RGB_QE21: CON3.R5, R12.3P
- new net RGB_QE22: CON3.R6, R12.2P
- new net RGB_QE23: CON3.R7, R12.1P
- new net RGB_QE3: CON3.B3, R3.1P
- new net RGB_QE4: CON3.B4, R8.4P
- new net RGB_QE5: CON3.B5, R8.3P
- new net RGB_QE6: CON3.B6, R8.2P
- new net RGB_QE7: CON3.B7, R8.1P
- new net RGB_QE8: CON3.G0, R9.4P
- new net RGB_QE9: CON3.G1, R9.3P
- new net RGB_VSYNC: CON3.VSYNC, R2.1P
- new net USB_D+: CON4.D+, IC7.D+
- new net USB_D-: CON4.D-, IC7.D-
- net +3V3: now also C13.P$2, C14.P$2, C4.P$2, C6.P$2, CON3.VCC, IC2.VOUT, IC5.AVDD@1, IC5.AVDD@2, IC5.AVDD@3, IC5.AVDD@4, IC5.DVDD@1, IC5.DVDD@2, IC5.DVDD@3, IC5.OVDD@1, IC5.OVDD@2, IC5.OVDD@3, IC5.OVDD@4, IC5.OVDD@5, IC5.PVDD, IC5.RSVD, R15.P$2, R4.P$2, R5.P$2, R6.P$2; no longer IC2.OUT, IC2.OUT1
- net GND: now also C10.P$1, C11.P$1, C13.P$1, C14.P$1, C3.P$2, C4.P$1, C5.P$2, C6.P$1, C7.P$1, C8.P$1, C9.P$2, CON1.2, CON1.3, CON2.CLKS, CON2.DATA0S, CON2.DATA1S, CON2.DATA2S, CON2.GND, CON2.GND@1, CON2.GND@2, CON2.GND@3, CON2.GND@4, CON3.GND@1, CON3.GND@2, CON3.GND@3, CON3.GND@4, CON3.GND@5, CON3.LED-K, CON4.GND@1, CON4.GND@2, CON4.GND@3, CON4.GND@4, CON4.GND@5, CON5.GND, CON5.GND@1, CON5.GND@2, IC1.GND, IC1.PGND, IC2.PGND, IC4.A0, IC4.A1, IC4.A2, IC4.GND, IC5.!STAG, IC5.AGND@1, IC5.AGND@2, IC5.AGND@3, IC5.AGND@4, IC5.AGND@5, IC5.DFO, IC5.DGND@1, IC5.DGND@2, IC5.DGND@3, IC5.OGND@1, IC5.OGND@2, IC5.OGND@3, IC5.OGND@4, IC5.OGND@5, IC5.PGND, IC7.GND@1, IC7.GND@2, IC7.GND@3, IC7.GND@4, IC7.UGND, JP1.1, JP2.1, JP3.1, JP4.1, JP5.1, R1.P$1, R14.P$2; no longer IC1.-
- net N$5: now also JP2.3, R5.P$1; no longer C1.P$1, IC1.+, IC2.IN
Other:
- note added: "+1.8V"
- note added: "+12V"
- note added: "+3.3V"
- note added: "+5V"
- note added: "21.03.2014"
- note added: "ATmega48"
- note added: "Atmel ATmega32U4"
- note added: "FT232RL"
- note added: "HDMI Connector"
- note added: "I2C EEPROM"
- note added: "LVDS-Display"
- note added: "POWER SUPPLY"
- note added: "S3: Spannungsversorgung +3.3V angepasst, Versorgungen hinzugefuegt (+5V, +9.6V, +12V), S4: HDMI Stecker, TFP401 und RGB Stecker hinzugefuegt"
- note added: "TFP401A"
- note added: "TODO: EN Pin auf Potential legen"
- note removed: "Atmel ATmega48"
- note removed: "RS232-USB-Bridge FTDI FT232RL"
- note removed: "UART"
- moved on the sheet: C1, C2, CON1

Commit message: end of workday 22.03.2014
Parts:
- added C12: 100n, SchlegelAr_Master:C_SMD0603
- added C15, C17, C19, C21, C22: 0.01u, SchlegelAr_Master:C_SMD0603
- added C16, C18, C20: 0.1u, SchlegelAr_Master:C_SMD0603
- added CON6: FI-X30SSLA-HF, SchlegelAr_Master:FI-X30SSLA-HF
- added IC6: ATMEGA48A-AU, SchlegelAr_Master:ATMEGA48A-AU
- added IC8: SN75LVDS83BDGGR, SchlegelAr_Master:SN75LVDS83BDGGR
- added JP6: JUMPER2THROUGHHOLE_2.54MM, SchlegelAr_Master:JUMPER2THROUGHHOLE_2.54MM
- added JP7, JP8: JUMPER3, SchlegelAr_Master:JUMPER3
- added R18: 10k, SchlegelAr_Master:R0603
- C11: value 1u -> 100n
- IC7: value ATMEGA32U4-AU -> FT232RL; device SchlegelAr_Master:ATMEGA32U4-AU -> SchlegelAr_Master:FT232RL
Connections:
- net N$41 renamed EDID_WRITEPROTECT
- removed net N$46: C8.P$2, IC7.XTAL1, Q1.1
- removed net N$47: C7.P$2, IC7.XTAL2, Q1.2
- removed net N$51: C11.P$2, IC7.UCAP
- removed net RGB_QE0: CON3.B0, R3.4P
- removed net RGB_QE1: CON3.B1, R3.3P
- removed net RGB_QE10: CON3.G2, R9.2P
- removed net RGB_QE11: CON3.G3, R9.1P
- removed net RGB_QE12: CON3.G4, R10.4P
- removed net RGB_QE13: CON3.G5, R10.3P
- removed net RGB_QE14: CON3.G6, R10.2P
- removed net RGB_QE15: CON3.G7, R10.1P
- removed net RGB_QE16: CON3.R0, R11.4P
- removed net RGB_QE17: CON3.R1, R11.3P
- removed net RGB_QE18: CON3.R2, R11.2P
- removed net RGB_QE19: CON3.R3, R11.1P
- removed net RGB_QE2: CON3.B2, R3.2P
- removed net RGB_QE20: CON3.R4, R12.4P
- removed net RGB_QE21: CON3.R5, R12.3P
- removed net RGB_QE22: CON3.R6, R12.2P
- removed net RGB_QE23: CON3.R7, R12.1P
- removed net RGB_QE3: CON3.B3, R3.1P
- removed net RGB_QE4: CON3.B4, R8.4P
- removed net RGB_QE5: CON3.B5, R8.3P
- removed net RGB_QE6: CON3.B6, R8.2P
- removed net RGB_QE7: CON3.B7, R8.1P
- removed net RGB_QE8: CON3.G0, R9.4P
- removed net RGB_QE9: CON3.G1, R9.3P
- new net AVR_PWM: IC6.PB1(OC1A/PCINT1), JP8.2
- new net AVR_XTAL1: C7.P$2, IC6.PB6(PCINT6/XTAL1/TOSC1), Q1.2
- new net AVR_XTAL2: C8.P$2, IC6.PB7(PCINT7/XTAL2/TOSC2), Q1.1
- new net FTDI_3V3OUT: C11.P$1, IC7.3V3OUT, IC7.VCCIO
- new net FTDI_RXD: IC6.(PDPCINT17/TXD)PD1, IC7.RXD
- new net FTDI_TXD: IC6.(PCINT16/RXD)PD0, IC7.TXD
- new net LVDS_0+: CON6.RA+, IC8.Y0P
- new net LVDS_0-: CON6.RA-, IC8.Y0M
- new net LVDS_1+: CON6.RB+, IC8.Y1P
- new net LVDS_1-: CON6.RB-, IC8.Y1M
- new net LVDS_2+: CON6.RC+, IC8.Y2P
- new net LVDS_2-: CON6.RC-, IC8.Y2M
- new net LVDS_3+: CON6.RDM+, IC8.Y3P
- new net LVDS_3-: CON6.RDM-, IC8.Y3M
- new net LVDS_CLK+: CON6.RCLK+, IC8.CLKOUTP
- new net LVDS_CLK-: CON6.RCLK-, IC8.CLKOUTM
- new net LVDS_PWM: CON6.PWM, JP8.3
- new net LVDS_REVSCAN: CON6.SHLI, JP7.2
- new net N$37: CON3.LED-A, JP6.2
- new net N$38: JP7.3, R18.P$1
- new net N$40: CON6.LED_EN
- new net RGB_EVEN_B0: CON3.B0, IC8.D15, R3.4P
- new net RGB_EVEN_B1: CON3.B1, IC8.D18, R3.3P
- new net RGB_EVEN_B2: CON3.B2, IC8.D19, R3.2P
- new net RGB_EVEN_B3: CON3.B3, IC8.D20, R3.1P
- new net RGB_EVEN_B4: CON3.B4, IC8.D21, R8.4P
- new net RGB_EVEN_B5: CON3.B5, IC8.D22, R8.3P
- new net RGB_EVEN_B6: CON3.B6, IC8.D16, R8.2P
- new net RGB_EVEN_B7: CON3.B7, IC8.D17, R8.1P
- new net RGB_EVEN_G0: CON3.G0, IC8.D7, R9.4P
- new net RGB_EVEN_G1: CON3.G1, IC8.D8, R9.3P
- new net RGB_EVEN_G2: CON3.G2, IC8.D9, R9.2P
- new net RGB_EVEN_G3: CON3.G3, IC8.D12, R9.1P
- new net RGB_EVEN_G4: CON3.G4, IC8.D13, R10.4P
- new net RGB_EVEN_G5: CON3.G5, IC8.D14, R10.3P
- new net RGB_EVEN_G6: CON3.G6, IC8.D10, R10.2P
- new net RGB_EVEN_G7: CON3.G7, IC8.D11, R10.1P
- new net RGB_EVEN_R0: CON3.R0, IC8.D0, R11.4P
- new net RGB_EVEN_R1: CON3.R1, IC8.D1, R11.3P
- new net RGB_EVEN_R2: CON3.R2, IC8.D2, R11.2P
- new net RGB_EVEN_R3: CON3.R3, IC8.D3, R11.1P
- new net RGB_EVEN_R4: CON3.R4, IC8.D4, R12.4P
- new net RGB_EVEN_R5: CON3.R5, IC8.D6, R12.3P
- new net RGB_EVEN_R6: CON3.R6, IC8.D27, R12.2P
- new net RGB_EVEN_R7: CON3.R7, IC8.D5, R12.1P
- new net RGB_PWM: JP8.1
- net +12V: now also CON6.VLED@1, CON6.VLED@2, CON6.VLED@3
- net +3V3: now also C15.P$2, C16.P$2, C17.P$2, C18.P$2, C19.P$2, C20.P$2, C21.P$2, C22.P$2, CON6.VCC@1, CON6.VCC@2, IC8.IOVCC@1, IC8.IOVCC@2, IC8.LVDSVCC, IC8.PLLVCC, IC8.VCC, R18.P$2
- net +5V: now also C12.P$1, IC6.AVCC, IC6.VCC@1, IC6.VCC@2, IC7.!RESET, IC7.VCC; no longer IC7.AREF, IC7.AVCC@1, IC7.AVCC@2, IC7.UVCC, IC7.VBUS, IC7.VCC@1, IC7.VCC@2
- net +9V6: now also JP6.1; no longer CON3.LED-A
- net AVR_!RESET: now also IC6.PC6(PCINT14/RESET); no longer IC7.!RESET
- net AVR_MISO: now also IC6.PB4(MISO/PCINT4)
- net AVR_MOSI: now also IC6.PB3(MOSI/OC2A/PCINT3)
- net AVR_SCK: now also IC6.PB5(SCK/PCINT5)
- net EDID_SCL: now also IC6.PC5(SCL/ADC5/PCINT13); no longer IC7.PD0(INT0/OC0B/SCL)
- net EDID_SDA: now also IC6.PC4(SDA/ADC4/PCINT12); no longer IC7.PD1(INT1/SDA)
- net GND: now also C11.P$2, C12.P$2, C15.P$1, C16.P$1, C17.P$1, C18.P$1, C19.P$1, C20.P$1, C21.P$1, C22.P$1, CON6.GND@1, CON6.GND@10, CON6.GND@11, CON6.GND@12, CON6.GND@13, CON6.GND@2, CON6.GND@3, CON6.GND@4, CON6.GND@5, CON6.GND@6, CON6.GND@7, CON6.GND@8, CON6.GND@9, IC6.GND@1, IC6.GND@2, IC6.GND@3, IC7.GND, IC7.GND@A, IC7.TEST, IC8.D23, IC8.GND@1, IC8.GND@10, IC8.GND@2, IC8.GND@3, IC8.GND@4, IC8.GND@5, IC8.GND@6, IC8.GND@7, IC8.GND@8, IC8.GND@9, JP7.1; no longer C11.P$1, IC7.GND@3, IC7.GND@4, IC7.UGND
- net RGB_DE: now also IC8.D26
- net RGB_HSYNC: now also IC8.D24
- net RGB_ODCK: now also IC8.CLKIN
- net RGB_VSYNC: now also IC8.D25
- net USB_D+: now also IC7.USBDM; no longer IC7.D+
- net USB_D-: now also IC7.USBDP; no longer IC7.D-
Other:
- note added: "22.03.2014"
- note added: "S5: EEPROM, ATMega48, FT232RL, USB und AVR_ISP Stecker hinzugefuegt, S6: SN75LVDS83 und LVDS Stecker hinzugefuegt"
- note added: "TODO: LED-A FET connect with AVR_PWM"
- note added: "TODO: LED_EN signal connect to AVR or Jumper"
- note removed: "TODO: EN Pin auf Potential legen"
- moved on the sheet: C10, C11, C7, C8, C9, CON3, CON4, CON5, IC4, JP5, Q1, R16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
