File: HDMI_RGB_Bridge/eagle/HDMI_RGB_LVDS/HDMI_RGB_LVDS.sch (EAGLE design)
At the start: 71 parts, among them CON1 KLDX-0202-A-LT, CON2 FCI-10029449-111RLF, CON3 XF2M-4015-1A, CON4 FCI-10033526-N3212LF, CON5 MOLEX-53261-0671, CON6 FI-X30SSLA-HF, IC1 WPMDL1300501BD, IC2 WPMDL1300331BD, IC3 TLV1117CDCYR, IC4 AT24C01C-SSHM-B, IC5 TFP401APZP, IC6 ATMEGA48A-AU, IC7 FT232RL, IC8 SN75LVDS83BDGGR, Q1 ATS073ASM-1, T1 IRF9530NSTRRPBF

Commit message: commit mid 24.03.2014
Parts:
- added C23, C24: 100n, SchlegelAr_Master:C_SMD0402
- added R19: 10k, SchlegelAr_Master:35WR5KLFTR
- added R20, R21: 140R, SchlegelAr_Master:R2512
- added SP1, SP10, SP11, SP12, SP13, SP14, SP15, SP16, SP17, SP18, SP2, SP3, SP4, SP5, SP9, U$95, U$96, U$97: SP2, SchlegelAr_Master:SP2
- added T2: IRLML2502TRPBF, SchlegelAr_Master:IRLML2502TRPBF
- C10, C11, C12, C13, C14, C15, C16, C17, C18, C19, C20, C21, C22, C4, C6, C7, C8, C9: device SchlegelAr_Master:C_SMD0603 -> SchlegelAr_Master:C_SMD0402
- JP1, JP2, JP3, JP7, JP8: value JUMPER3 -> JUMPER2; device SchlegelAr_Master:JUMPER3 -> SchlegelAr_Master:JUMPER2
- JP5: value JUMPER2THROUGHHOLE_2.54MM -> JUMPER2; device SchlegelAr_Master:JUMPER2THROUGHHOLE_2.54MM -> SchlegelAr_Master:JUMPER2
- JP6: value JUMPER2THROUGHHOLE_2.54MM -> JUMPER3; device SchlegelAr_Master:JUMPER2THROUGHHOLE_2.54MM -> SchlegelAr_Master:JUMPER3
- R1, R13, R14, R15, R16, R17, R18, R4, R5, R6, R7: device SchlegelAr_Master:R0603 -> SchlegelAr_Master:R0402
Connections:
- net EDID_WRITEPROTECT renamed EDID_WP
- removed net HDMI_ST: IC5.ST, JP3.2
- removed net N$10: JP1.3, R6.P$1
- removed net N$3: JP3.3, R4.P$1
- removed net N$36: JP4.3, R15.P$1
- removed net N$38: JP7.3, R18.P$1
- removed net N$40: CON6.LED_EN
- removed net N$5: JP2.3, R5.P$1
- new net AVR_PWM_ADC: IC6.PC0(ADC0/PCINT8), R19.S
- new net LVDS_LED_EN: CON6.LED_EN, JP8.2, R4.P$1
- new net N$39: C22.P$2, IC8.IOVCC@1, SP15.1
- new net N$41: C21.P$2, IC8.IOVCC@2, SP16.1
- new net N$42: C15.P$2, C18.P$2, IC8.LVDSVCC, SP17.1
- new net N$43: C19.P$2, C20.P$2, IC8.PLLVCC, SP18.1
- new net N$44: C12.P$1, IC7.VCC, SP9.1
- new net N$45: C24.P$1, IC6.AVCC, SP13.2
- new net N$46: C9.P$1, IC6.VCC@1, SP11.2
- new net N$47: C23.P$1, IC6.VCC@2, SP12.2
- new net N$48: C16.P$2, C17.P$2, IC8.VCC, SP14.1
- new net N$49: C10.P$2, IC4.VCC, SP10.2
- new net N$50: C6.P$2, IC5.OVDD@1, IC5.OVDD@2, IC5.OVDD@3, IC5.OVDD@4, IC5.OVDD@5, SP4.1
- new net N$51: C2.P$1, U$96.1
- new net N$52: C4.P$2, IC5.AVDD@1, IC5.AVDD@2, IC5.AVDD@3, IC5.AVDD@4, SP5.1
- new net N$53: C13.P$2, IC5.PVDD, SP2.1
- new net N$54: C14.P$2, IC5.DVDD@1, IC5.DVDD@2, IC5.DVDD@3, SP3.1
- new net N$55: C3.P$1, U$97.1
- new net N$56: C5.P$1, U$95.1
- new net N$57: R20.P$1, R21.P$1, T2.D
- new net N$59: C1.P$1, D1.C, IC1.VIN, IC2.VIN, IC3.IN, SP1.1, T1.S
- new net RGB_PWM_EN: JP4.2, T2.G
- net +12V: now also SP1.2; no longer C1.P$1, D1.C, IC1.VIN, IC2.VIN, IC3.IN, T1.S
- net +3V3: now also JP4.1, SP14.2, SP15.2, SP16.2, SP17.2, SP18.2, SP2.2, SP3.2, SP4.2, SP5.2, U$96.2; no longer C13.P$2, C14.P$2, C15.P$2, C16.P$2, C17.P$2, C18.P$2, C19.P$2, C2.P$1, C20.P$2, C21.P$2, C22.P$2, C4.P$2, C6.P$2, IC5.AVDD@1, IC5.AVDD@2, IC5.AVDD@3, IC5.AVDD@4, IC5.DVDD@1, IC5.DVDD@2, IC5.DVDD@3, IC5.OVDD@1, IC5.OVDD@2, IC5.OVDD@3, IC5.OVDD@4, IC5.OVDD@5, IC5.PVDD, IC8.IOVCC@1, IC8.IOVCC@2, IC8.LVDSVCC, IC8.PLLVCC, IC8.VCC
- net +5V: now also IC6.AREF, IC7.VCCIO, R19.E, SP10.1, SP11.1, SP12.1, SP13.1, SP9.2, U$95.2; no longer C10.P$2, C12.P$1, C5.P$1, C9.P$1, IC4.VCC, IC6.AVCC, IC6.VCC@1, IC6.VCC@2, IC7.VCC
- net +9V6: now also R20.P$2, R21.P$2, U$97.2; no longer C3.P$1, JP6.1
- net AVR_PWM: now also JP6.2; no longer JP8.2
- net FTDI_3V3OUT: no longer IC7.VCCIO
- net GND: now also C23.P$2, C24.P$2, IC5.ST, JP8.1, R19.A; no longer JP4.1
- net HDMI_OCK_INV: now also R6.P$1
- net HDMI_PIXS: now also R5.P$1
- net LVDS_PWM: now also JP6.3; no longer JP8.3
- net LVDS_REVSCAN: now also R18.P$1
- net N$37: now also T2.S; no longer JP6.2
- net RGB_DISP: now also JP3.2, R15.P$1; no longer JP4.2
- net RGB_PWM: now also JP4.3, JP6.1; no longer JP8.1
Other:
- note added: "24.03.2014"
- note added: "AVR_PWM"
- note added: "Default"
- note added: "Description"
- note added: "EDID_WP"
- note added: "Enables the RGB Display Jumper present: Display disabled No jumper: Display enabled"
- note added: "Erstellung des Projekts, S1: Blockschaltbild, Versorgungsgraph hinzugefuegt, S2: Blockschaltbild, S3: Spannungsversorgung +3.3V hinzugefuegt"
- note added: "HDMI_OCK_INV"
- note added: "HDMI_PIXS"
- note added: "JP 2-3"
- note added: "JP1"
- note added: "JP2"
- note added: "JP3"
- note added: "JP5"
- note added: "JP7"
- note added: "JP8"
- note added: "Jumper"
- note added: "Jumper present"
- note added: "LVDS_LED_EN"
- note added: "LVDS_REVSCAN"
- note added: "NOTE: AVCC as reference voltage for ADC"
- note added: "NOTE: LCD Backlight 9.6V@170mA => R = 70 Ohm, 2W"
- note added: "NOTE: VCCIO is +5V because AVR is +5V"
- note added: "NOTE: WPMDL1300331BD has internal pullup on EN-pin."
- note added: "NOTE: WPMDL1300501BD has internal pullup on EN-pin."
- note added: "No Jumper"
- note added: "No default"
- note added: "ODCK Polarity Selects ODCK edge on which pixel data and control signals are latched. Jumper present: Latches output data on falling ODCK edge No Jumper: Latches output data on rising ODCK edge"
- note added: "Pixelselect: Selects between one or two pixels per clock output modes. During the 2-pixel/clck mode, both even pixels and odd pixels, are output in tandem on a given clock cycle. During the 1-pixel/clock mode, even and odd pixels are output sequentially, on the same time, with the even pixel first, on the even pixel bus. Jumper present: 1-pixel/clock No Jumper: 2-pixel/clock"
- note added: "RGB_DISP"
- note added: "RGB_PWM_EN"
- note added: "S4: PWM Ansteuerung fuer RGB Display Hintergrundbeleuchtung hinzugefuegt, Jumper modifiziert, Tabelle fuer Jumpererklaerung hinzugefuegt S5: Potentiometer und ADC-Messung hinzugefuegt, Jumper modifiziert, Tabelle fuer Jumpererklaerung hinzugefuegt S6: Jumper modifiziert, Tabelle fuer Jumpererklaerung hinzugefuegt, alle: Sternpunkte eingebaut"
- note added: "Selects if the LVDS backlight is enabled Jumper present: backlight disabled No Jumper: backlight enabled"
- note added: "Selects the PWM output to the used display JP 1-2: RGB Display JP 2-3: LVDS Display"
- note added: "Selects the backlight mode for the RGB display: JP 1-2: Backlight turned on permanentely JP 2-3: Backlight controlled via PWM"
- note added: "Selects the scanning direction of the LVDS display Jumper present: Left->Right (Up->Down) No Jumper: Right->Left (Down->Up)"
- note added: "Selects the write protection mode for the I2C eeprom Jumper present: write protection enabled No Jumper: write protection disabled"
- note added: "Signal"
- note removed: "Erstellung des Projekts, S2: Blockschaltbild, S3: Spannungsversorgung +3.3V hinzugefuegt"
- note removed: "TODO: LED-A FET connect with AVR_PWM"
- note removed: "TODO: LED_EN signal connect to AVR or Jumper"
- moved on the sheet: C1, C10, C12, C13, C14, C15, C16, C17, C18, C2, C21, C22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

Commit message: end of workday 24.03.2014
Parts:
- added R22, R23: 0R, SchlegelAr_Master:R0402
Connections:
- new net N$10: IC7.USBDM, R23.P$2
- new net N$5: IC7.USBDP, R22.P$2
- net USB_D+: now also R23.P$1; no longer IC7.USBDM
- net USB_D-: now also R22.P$1; no longer IC7.USBDP
Changed lines of the file:
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@@
 <part name="SP18" library="SchlegelAr_Master" deviceset="SP2" device=""/>
 <part name="U$35" library="SchlegelAr_Master" deviceset="+5V" device=""/>
+<part name="R22" library="SchlegelAr_Master" deviceset="R" device="0402" value="0R"/>
+<part name="R23" library="SchlegelAr_Master" deviceset="R" device="0402" value="0R"/>
 </parts>
 <sheets>
@@
 <instance part="SP13" gate="G$1" x="152.4" y="182.88"/>
 <instance part="U$35" gate="G$1" x="142.24" y="195.58"/>
+<instance part="R22" gate="G$1" x="76.2" y="200.66"/>
+<instance part="R23" gate="G$1" x="86.36" y="198.12"/>
 </instances>
 <busses>
@@
 </segment>
 <segment>
-<wire x1="99.06" y1="200.66" x2="86.36" y2="200.66" width="0.1524" layer="91"/>
-<label x="86.36" y="200.66" size="1.27" layer="95" rot="R180" xref="yes"/>
-<pinref part="IC7" gate="G$1" pin="USBDP"/>
+<label x="68.58" y="200.66" size="1.27" layer="95" rot="R180" xref="yes"/>
+<wire x1="71.12" y1="200.66" x2="68.58" y2="200.66" width="0.1524" layer="91"/>
+<pinref part="R22" gate="G$1" pin="P$1"/>
 </segment>
 </net>
@@
 </segment>
 <segment>
-<wire x1="99.06" y1="198.12" x2="86.36" y2="198.12" width="0.1524" layer="91"/>
-<label x="86.36" y="198.12" size="1.27" layer="95" rot="R180" xref="yes"/>
-<pinref part="IC7" gate="G$1" pin="USBDM"/>
+<label x="68.58" y="198.12" size="1.27" layer="95" rot="R180" xref="yes"/>
+<wire x1="81.28" y1="198.12" x2="68.58" y2="198.12" width="0.1524" layer="91"/>
+<pinref part="R23" gate="G$1" pin="P$1"/>
 </segment>
 </net>
@@
 </segment>
 </net>
+<net name="N$5" class="0">
+<segment>
+<pinref part="R22" gate="G$1" pin="P$2"/>
+<pinref part="IC7" gate="G$1" pin="USBDP"/>
+<wire x1="81.28" y1="200.66" x2="99.06" y2="200.66" width="0.1524" layer="91"/>
+</segment>
+</net>
+<net name="N$10" class="0">
+<segment>
+<pinref part="IC7" gate="G$1" pin="USBDM"/>
+<pinref part="R23" gate="G$1" pin="P$2"/>
+<wire x1="99.06" y1="198.12" x2="91.44" y2="198.12" width="0.1524" layer="91"/>
+</segment>
+</net>
