File: HDMI_RGB_Bridge/eagle/HDMI_RGB_LVDS/HDMI_RGB_LVDS.bak.brd (EAGLE design)
At the start: 90 x 60 mm, 81 parts, among them CON1 KLDX-0202-A-LT, CON2 FCI-10029449-111RLF, CON3 XF2M-4015-1A, CON4 FCI-10033526-N3212LF, CON5 MOLEX-53261-0671, CON6 FI-X30SSLA-HF, IC1 WPMDL1300501BD, IC2 WPMDL1300331BD, IC3 TLV1117CDCYR, IC4 AT24C01C-SSHM-B, IC5 TFP401APZP, IC6 ATMEGA48A-AU, IC7 FT232RL, IC8 SN75LVDS83BDGGR, Q1 ATS073ASM-1, T1 IRF9530NSTRRPBF, T2 IRLML2502TRPBF

Commit message: uploaded finished schematic and layout
Parts:
- moved R3 14.9 mm to (48.6, 41.4), turned to 180 degrees
- moved R10 12.5 mm to (32.1, 40.8), turned to 180 degrees
- moved R11 7.13 mm to (32.1, 37.4), turned to 180 degrees
- moved R8 6.92 mm to (48.6, 38.2), turned to 180 degrees
- moved R12 2.51 mm to (32.1, 33.9), turned to 180 degrees
- moved R2 2.22 mm to (32.1, 30.5), turned to 180 degrees
- moved R9 2.08 mm to (48.6, 34.9), turned to 180 degrees
- moved C22 1.75 mm to (21.2, 47.6)
- moved C13 1.08 mm to (50.7, 22.6), turned to 45 degrees
- moved R18 0.14 mm to (11.5, 17.6), turned to 90 degrees
Routing:
- net +12V: track 45.5 -> 143.9 mm
- net RGB_PWM_EN: track 0.00 -> 64.9 mm, vias 0 -> 2
- net RGB_DISP: track 2.25 -> 61.4 mm
- net LVDS_REVSCAN: track 2.25 -> 43.9 mm, vias 0 -> 3
- net EDID_SDA: track 10.8 -> 52.2 mm, vias 1 -> 2
- net GND: track 110.8 -> 149.7 mm, vias 78 -> 111
- net EDID_SCL: track 12.4 -> 48.6 mm, vias 1 -> 2
- net N$13: track 0.00 -> 27.0 mm, vias 0 -> 2
- net LVDS_PWM: track 0.00 -> 26.2 mm, vias 0 -> 1
- net N$12: track 0.00 -> 25.3 mm, vias 0 -> 2
- net N$11: track 0.00 -> 23.6 mm, vias 0 -> 2
- net N$9: track 0.00 -> 21.9 mm, vias 0 -> 2
- net +3V3: track 34.0 -> 55.1 mm, vias 7 -> 25
- net N$17: track 0.00 -> 20.2 mm, vias 0 -> 2
- net N$26: track 0.00 -> 18.8 mm
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- added copper zone on layer 15, net +3V3
