File: HDMI_RGB_Bridge/eagle/HDMI_RGB_LVDS/HDMI_RGB_LVDS_fertig_V1.brd (EAGLE design)
At the start: 90 x 60 mm, 81 parts, among them CON1 KLDX-0202-A-LT, CON2 FCI-10029449-111RLF, CON3 XF2M-4015-1A, CON4 FCI-10033526-N3212LF, CON5 MOLEX-53261-0671, CON6 FI-X30SSLA-HF, IC1 WPMDL1300501BD, IC2 WPMDL1300331BD, IC3 TLV1117CDCYR, IC4 AT24C01C-SSHM-B, IC5 TFP401APZP, IC6 ATMEGA48A-AU, IC7 FT232RL, IC8 SN75LVDS83BDGGR, Q1 ATS073ASM-1, T1 IRF9530NSTRRPBF, T2 IRLML2502TRPBF

Commit message: uploaded finished schematic and layout
Parts:
- removed SP10, SP9: SP2, SchlegelAr_Master:SP2
- moved R3 14.9 mm to (48.6, 41.4), turned to 180 degrees
- moved U$1 12.7 mm to (0.05, 0.06)
- moved R10 12.5 mm to (32.1, 40.8), turned to 180 degrees
- moved R11 7.13 mm to (32.1, 37.4), turned to 180 degrees
- moved R8 6.92 mm to (48.6, 38.2), turned to 180 degrees
- moved R23 3.70 mm to (2.75, 7.19), turned to 90 degrees
- moved R12 2.51 mm to (32.1, 33.9), turned to 180 degrees
- moved C11 2.38 mm to (6.81, 12.8)
- moved R22 2.31 mm to (1.44, 7.19), turned to 90 degrees
- moved R18 2.29 mm to (13.4, 18.8), turned to 90 degrees
- moved C10 2.22 mm to (17.5, 8.94)
- moved C12 2.22 mm to (8.62, 13.8)
- moved C23 2.22 mm to (27.1, 11.7)
- moved C24 2.22 mm to (14.1, 12.4)
- moved C7 2.22 mm to (28.5, 12.3)
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Connections:
- net LVDS_0+ renamed LVDS_0_P
- net LVDS_0- renamed LVDS_0_N
- net LVDS_1+ renamed LVDS_1_P
- net LVDS_1- renamed LVDS_1_N
- net LVDS_2+ renamed LVDS_2_P
- net LVDS_2- renamed LVDS_2_N
- net LVDS_3+ renamed LVDS_3_P
- net LVDS_3- renamed LVDS_3_N
- net LVDS_CLK+ renamed LVDS_CLK_P
- net LVDS_CLK- renamed LVDS_CLK_N
- removed net N$44: C12.1, IC7.20, SP9.P$1
- removed net N$49: C10.2, IC4.8, SP10.P$2
- net +5V: now also C10.2, C12.1, IC4.8, IC7.20; no longer SP10.P$1, SP9.P$2
Routing:
- net +12V: track 45.5 -> 145.5 mm
- net RGB_EVEN_R2: track 0.00 -> 73.0 mm, vias 0 -> 3
- net RGB_EVEN_R4: track 0.00 -> 67.8 mm, vias 0 -> 2
- net RGB_EVEN_G3: track 0.00 -> 66.2 mm, vias 0 -> 4
- net RGB_EVEN_R6: track 0.00 -> 63.8 mm, vias 0 -> 3
- net RGB_PWM_EN: track 0.00 -> 62.5 mm, vias 0 -> 2
- net RGB_EVEN_R1: track 0.00 -> 59.7 mm, vias 0 -> 5
- net RGB_EVEN_G0: track 0.00 -> 59.2 mm, vias 0 -> 4
- net RGB_DISP: track 2.25 -> 61.4 mm
- net RGB_EVEN_R3: track 0.00 -> 58.2 mm, vias 0 -> 4
- net RGB_EVEN_G1: track 0.00 -> 58.0 mm, vias 0 -> 4
- net RGB_EVEN_G2: track 0.00 -> 57.9 mm, vias 0 -> 4
- net RGB_EVEN_B1: track 0.00 -> 57.7 mm, vias 0 -> 3
- net RGB_EVEN_B2: track 0.00 -> 52.9 mm, vias 0 -> 3
- net RGB_EVEN_R0: track 0.00 -> 51.8 mm, vias 0 -> 4
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- added copper zone on layer 15, net +3V3
- added copper zone on layer 1, net GND
- added copper zone on layer 16, net GND
Other:
- board text added: "1"
- board text added: "2"
- board text added: "25.03.2014"
- board text added: "3"
- board text added: "4"
- board text added: "Armin Schlegel"
- board text added: "HDMI_RGB_LVDS V1"
