File: HDMI_RGB_Bridge/eagle/HDMI_RGB_LVDS/HDMI_RGB_LVDS_fertig_V1.sch (EAGLE design)
At the start: 95 parts, among them CON1 KLDX-0202-A-LT, CON2 FCI-10029449-111RLF, CON3 XF2M-4015-1A, CON4 FCI-10033526-N3212LF, CON5 MOLEX-53261-0671, CON6 FI-X30SSLA-HF, IC1 WPMDL1300501BD, IC2 WPMDL1300331BD, IC3 TLV1117CDCYR, IC4 AT24C01C-SSHM-B, IC5 TFP401APZP, IC6 ATMEGA48A-AU, IC7 FT232RL, IC8 SN75LVDS83BDGGR, Q1 ATS073ASM-1, T1 IRF9530NSTRRPBF, T2 IRLML2502TRPBF

Commit message: uploaded finished schematic and layout
Parts:
- removed SP1, SP10, SP11, SP12, SP13, SP14, SP15, SP16, SP17, SP18, SP2, SP3, SP4, SP5, SP9, U$97: SP2, SchlegelAr_Master:SP2
Connections:
- net LVDS_0+ renamed LVDS_0_P
- net LVDS_0- renamed LVDS_0_N
- net LVDS_1+ renamed LVDS_1_P
- net LVDS_1- renamed LVDS_1_N
- net LVDS_2+ renamed LVDS_2_P
- net LVDS_2- renamed LVDS_2_N
- net LVDS_3+ renamed LVDS_3_P
- net LVDS_3- renamed LVDS_3_N
- net LVDS_CLK+ renamed LVDS_CLK_P
- net LVDS_CLK- renamed LVDS_CLK_N
- removed net N$39: C22.P$2, IC8.IOVCC@1, SP15.1
- removed net N$41: C21.P$2, IC8.IOVCC@2, SP16.1
- removed net N$42: C15.P$2, C18.P$2, IC8.LVDSVCC, SP17.1
- removed net N$43: C19.P$2, C20.P$2, IC8.PLLVCC, SP18.1
- removed net N$44: C12.P$1, IC7.VCC, SP9.1
- removed net N$45: C24.P$1, IC6.AVCC, SP13.2
- removed net N$46: C9.P$1, IC6.VCC@1, SP11.2
- removed net N$47: C23.P$1, IC6.VCC@2, SP12.2
- removed net N$48: C16.P$2, C17.P$2, IC8.VCC, SP14.1
- removed net N$49: C10.P$2, IC4.VCC, SP10.2
- removed net N$50: C6.P$2, IC5.OVDD@1, IC5.OVDD@2, IC5.OVDD@3, IC5.OVDD@4, IC5.OVDD@5, SP4.1
- removed net N$52: C4.P$2, IC5.AVDD@1, IC5.AVDD@2, IC5.AVDD@3, IC5.AVDD@4, SP5.1
- removed net N$53: C13.P$2, IC5.PVDD, SP2.1
- removed net N$54: C14.P$2, IC5.DVDD@1, IC5.DVDD@2, IC5.DVDD@3, SP3.1
- removed net N$55: C3.P$1, U$97.1
- removed net N$59: C1.P$1, D1.C, IC1.VIN, IC2.VIN, IC3.IN, SP1.1, T1.S
- net +12V: now also C1.P$1, D1.C, IC1.VIN, IC2.VIN, IC3.IN, T1.S; no longer SP1.2
- net +3V3: now also C13.P$2, C14.P$2, C15.P$2, C16.P$2, C17.P$2, C18.P$2, C19.P$2, C20.P$2, C21.P$2, C22.P$2, C4.P$2, C6.P$2, IC5.AVDD@1, IC5.AVDD@2, IC5.AVDD@3, IC5.AVDD@4, IC5.DVDD@1, IC5.DVDD@2, IC5.DVDD@3, IC5.OVDD@1, IC5.OVDD@2, IC5.OVDD@3, IC5.OVDD@4, IC5.OVDD@5, IC5.PVDD, IC8.IOVCC@1, IC8.IOVCC@2, IC8.LVDSVCC, IC8.PLLVCC, IC8.VCC; no longer SP14.2, SP15.2, SP16.2, SP17.2, SP18.2, SP2.2, SP3.2, SP4.2, SP5.2
- net +5V: now also C10.P$2, C12.P$1, C23.P$1, C24.P$1, C9.P$1, IC4.VCC, IC6.AVCC, IC6.VCC@1, IC6.VCC@2, IC7.VCC; no longer SP10.1, SP11.1, SP12.1, SP13.1, SP9.2
- net +9V6: now also C3.P$1; no longer U$97.2
Other:
- note added: "+9.6V"
- note added: "25.03.2014"
- note added: "AVR"
- note added: "AVR ISP connector"
- note added: "EDID EEPROM"
- note added: "FTDI FT232RL"
- note added: "HDMI connector"
- note added: "HDMI to RGB bridge"
- note added: "LVDS display connector"
- note added: "LVDS-Display backlight"
- note added: "Power Supply"
- note added: "RGB Display connector"
- note added: "RGB to LVDS bridge"
- note added: "RGB-Display backlight"
- note added: "S2: Blockschaltbild angepasst, Versorgungsgraph angepasst"
- note added: "S4: PWM Ansteuerung fuer RGB Display Hintergrundbeleuchtung hinzugefuegt, Jumper modifiziert, Tabelle fuer Jumpererklaerung hinzugefuegt S5: Potentiometer und ADC-Messung hinzugefuegt, Jumper modifiziert, Tabelle fuer Jumpererklaerung hinzugefuegt S6: Jumper modifiziert, Tabelle fuer Jumpererklaerung hinzugefuegt"
- note added: "SN75LVDS83B"
- note added: "UART"
- note added: "USB UART Bridge"
- note added: "USB connector"
- note removed: "+1.8V"
- note removed: "HDMI Connector"
- note removed: "LVDS-Display"
- note removed: "POWER SUPPLY"
- note removed: "S4: PWM Ansteuerung fuer RGB Display Hintergrundbeleuchtung hinzugefuegt, Jumper modifiziert, Tabelle fuer Jumpererklaerung hinzugefuegt S5: Potentiometer und ADC-Messung hinzugefuegt, Jumper modifiziert, Tabelle fuer Jumpererklaerung hinzugefuegt S6: Jumper modifiziert, Tabelle fuer Jumpererklaerung hinzugefuegt, alle: Sternpunkte eingebaut"
- moved on the sheet: C10, C11, C12, C23, C24, C7, C8, C9, CON3, CON4, CON5, IC4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
