File: HDMI_RGB_Bridge/eagle/HDMI_RGB_LVDS/HDMI_RGB_LVDS_fertig_V4.brd (EAGLE design)
At the start: 90 x 60 mm, 79 parts, among them CON1 KLDX-0202-A-LT, CON2 FCI-10029449-111RLF, CON3 XF2M-4015-1A, CON4 FCI-10033526-N3212LF, CON5 MOLEX-53261-0671, CON6 FI-X30SSLA-HF, IC1 WPMDL1300501BD, IC2 WPMDL1300331BD, IC3 TLV1117CDCYR, IC4 AT24C01C-SSHM-B, IC5 TFP401APZP, IC6 ATMEGA48A-AU, IC7 FT232RL, IC8 SN75LVDS83BDGGR, Q1 ATS073ASM-1, T1 IRF9530NSTRRPBF, T2 IRLML2502TRPBF

Commit message: updated V4 of layout
Parts:
- moved R1 1.69 mm to (88.6, 30.4)
- moved Q1 1.19 mm to (31.7, 12.4)
Routing:
- net GND: track 156.0 -> 152.3 mm
- net +3V3: track 56.9 -> 54.1 mm, vias 25 -> 27
- net AVR_XTAL2: track 10.6 -> 8.91 mm
- net AVR_XTAL1: track 10.4 -> 11.3 mm
- net N$4: track 7.48 -> 6.77 mm
- net LVDS_REVSCAN: track 41.6 -> 40.9 mm
- net INT_RGB_EVEN_B4: track 16.3 -> 15.8 mm
- net +5V: track 45.0 -> 44.6 mm, vias 12 -> 14
- added copper zone on layer 1, net +3V3
- added copper zone on layer 16, net +3V3
- added copper zone on layer 1, net +5V
- added copper zone on layer 16, net +5V
Other:
- board text added: "27.03.2014"
- board text removed: "26.03.2014"

Commit message: updated version of V4
Parts:
- added LED1, LED2, LED3, LED4: (no value), SchlegelAr_Master:LED0402
- added R24: 261R, SchlegelAr_Master:R0402
- added R25: 600R, SchlegelAr_Master:R0402
- added R26: 1k5, SchlegelAr_Master:R0402
- added R27: 2k5, SchlegelAr_Master:R0402
- C7, C8: value 10p -> 22p
Connections:
- new net N$1: LED1.A, R24.2
- new net N$6: LED2.A, R25.2
- new net N$7: LED3.A, R26.2
- new net N$8: LED4.A, R27.2
- net +12V: now also LED4.C
- net +3V3: now also LED2.C
- net +5V: now also LED1.C
- net +9V6: now also LED3.C
- net GND: now also R24.1, R25.1, R26.1, R27.1
Routing:
- net +5V: track 44.6 -> 74.4 mm, vias 14 -> 15
- net +3V3: track 54.1 -> 77.5 mm, vias 27 -> 28
- net +9V6: track 19.1 -> 27.4 mm, vias 0 -> 1
- net +12V: track 143.4 -> 148.8 mm
- net GND: track 152.3 -> 155.7 mm, vias 95 -> 99
- net N$7: track 0.00 -> 1.01 mm
- net N$6: track 0.00 -> 1.01 mm
- net N$8: track 0.00 -> 0.95 mm
- net N$1: track 0.00 -> 0.89 mm
Changed lines of the file:
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@@
 <layer number="3" name="Route3" color="4" fill="3" visible="no" active="no"/>
 <layer number="14" name="Route14" color="1" fill="6" visible="no" active="no"/>
-<layer number="15" name="Route15" color="4" fill="6" visible="no" active="yes"/>
+<layer number="15" name="Route15" color="4" fill="6" visible="yes" active="yes"/>
 <layer number="16" name="Bottom" color="1" fill="1" visible="yes" active="yes"/>
 <layer number="17" name="Pads" color="2" fill="1" visible="yes" active="yes"/>
 <layer number="18" name="Vias" color="2" fill="1" visible="yes" active="yes"/>
 <layer number="19" name="Unrouted" color="6" fill="1" visible="yes" active="yes"/>
-<layer number="20" name="Dimension" color="15" fill="1" visible="no" active="yes"/>
+<layer number="20" name="Dimension" color="15" fill="1" visible="yes" active="yes"/>
 <layer number="21" name="tPlace" color="7" fill="1" visible="no" active="yes"/>
 <layer number="22" name="bPlace" color="7" fill="1" visible="no" active="yes"/>
-<layer number="23" name="tOrigins" color="15" fill="1" visible="no" active="yes"/>
-<layer number="24" name="bOrigins" color="15" fill="1" visible="no" active="yes"/>
-<layer number="25" name="tNames" color="7" fill="1" visible="no" active="yes"/>
+<layer number="23" name="tOrigins" color="15" fill="1" visible="yes" active="yes"/>
+<layer number="24" name="bOrigins" color="15" fill="1" visible="yes" active="yes"/>
+<layer number="25" name="tNames" color="7" fill="1" visible="yes" active="yes"/>
 <layer number="26" name="bNames" color="7" fill="1" visible="no" active="yes"/>
 <layer number="27" name="tValues" color="7" fill="1" visible="no" active="yes"/>
@@
 <attribute name="VALUE" x="27.4965" y="18.09" size="1.27" layer="27" ratio="10" rot="R270"/>
 </element>
-<element name="C7" library="SchlegelAr_Master" package="C0402" value="10p" x="28.5" y="12.3125" smashed="yes" rot="R90">
+<element name="C7" library="SchlegelAr_Master" package="C0402" value="22p" x="28.5" y="12.3125" smashed="yes" rot="R90">
 <attribute name="NAME" x="29.0525" y="9.0525" size="1.27" layer="25" rot="R90"/>
 <attribute name="VALUE" x="30.405" y="11.6775" size="1.27" layer="27" rot="R90"/>
 </element>
-<element name="C8" library="SchlegelAr_Master" package="C0402" value="10p" x="28.5" y="14.5625" smashed="yes" rot="R270">
+<element name="C8" library="SchlegelAr_Master" package="C0402" value="22p" x="28.5" y="14.5625" smashed="yes" rot="R270">
 <attribute name="NAME" x="27.8225" y="18.135" size="1.27" layer="25" rot="R270"/>
 <attribute name="VALUE" x="26.595" y="15.1975" size="1.27" layer="27" rot="R270"/>
@@
 <attribute name="NAME" x="3.4275" y="8.3025" size="1.27" layer="25" rot="R90"/>
 <attribute name="VALUE" x="4.655" y="6.5525" size="1.27" layer="27" rot="R90"/>
+</element>
+<element name="LED1" library="SchlegelAr_Master" package="LED0402" value="" x="85.625" y="47.25" rot="R180"/>
+<element name="LED2" library="SchlegelAr_Master" package="LED0402" value="" x="85.5625" y="44.875" rot="R180"/>
+<element name="LED3" library="SchlegelAr_Master" package="LED0402" value="" x="85.5" y="42.25" rot="R180"/>
+<element name="LED4" library="SchlegelAr_Master" package="LED0402" value="" x="85.5625" y="39.6875" rot="R180"/>
+<element name="R24" library="SchlegelAr_Master" package="R0402" value="261R" x="87.8125" y="47.25" smashed="yes" rot="R180">
+<attribute name="NAME" x="89.9475" y="46.74" size="1.27" layer="25" rot="R180"/>
+<attribute name="VALUE" x="88.4475" y="49.155" size="1.27" layer="27" rot="R180"/>
+</element>
+<element name="R25" library="SchlegelAr_Master" package="R0402" value="600R" x="87.875" y="44.875" smashed="yes" rot="R180">
+<attribute name="NAME" x="89.9475" y="44.1775" size="1.27" layer="25" rot="R180"/>
+<attribute name="VALUE" x="88.51" y="46.78" size="1.27" layer="27" rot="R180"/>
+</element>
+<element name="R26" library="SchlegelAr_Master" package="R0402" value="1k5" x="87.8125" y="42.25" smashed="yes" rot="R180">
+<attribute name="NAME" x="89.9475" y="41.615" size="1.27" layer="25" rot="R180"/>
+<attribute name="VALUE" x="88.4475" y="44.155" size="1.27" layer="27" rot="R180"/>
+</element>
+<element name="R27" library="SchlegelAr_Master" package="R0402" value="2k5" x="87.8125" y="39.6875" smashed="yes" rot="R180">
+<attribute name="NAME" x="89.9475" y="39.0525" size="1.27" layer="25" rot="R180"/>
+<attribute name="VALUE" x="88.4475" y="41.5925" size="1.27" layer="27" rot="R180"/>
 </element>
 </elements>
@@
 <wire x1="2.36875" y1="22.85625" x2="4.14375" y2="22.85625" width="0.3" layer="16"/>
 <wire x1="4.14375" y1="22.85625" x2="4.1875" y2="22.8125" width="0.3" layer="16"/>
+<contactref element="R24" pad="1"/>
+<contactref element="R25" pad="1"/>
+<contactref element="R26" pad="1"/>
+<contactref element="R27" pad="1"/>
+<wire x1="88.4625" y1="47.25" x2="89.3125" y2="47.25" width="0.3" layer="1"/>
+<wire x1="88.525" y1="44.875" x2="88.5875" y2="44.8125" width="0.3" layer="1"/>
+<wire x1="88.5875" y1="44.8125" x2="89.375" y2="44.8125" width="0.3" layer="1"/>
+<wire x1="88.4625" y1="42.25" x2="88.525" y2="42.1875" width="0.3" layer="1"/>
+<wire x1="88.525" y1="42.1875" x2="89.3125" y2="42.1875" width="0.3" layer="1"/>
+<wire x1="88.4625" y1="39.6875" x2="89.3125" y2="39.6875" width="0.3" layer="1"/>
+<via x="89.3125" y="42.1875" extent="1-16" drill="0.3"/>
+<via x="89.3125" y="39.6875" extent="1-16" drill="0.3"/>
+<via x="89.375" y="44.8125" extent="1-16" drill="0.3"/>
+<via x="89.3125" y="47.25" extent="1-16" drill="0.3"/>
 </signal>
 <signal name="+3V3">
@@
 <wire x1="46.8125" y1="16.1875" x2="46.8125" y2="15.625" width="0.3" layer="1"/>
 <wire x1="46.8125" y1="15.625" x2="47" y2="15.4375" width="0.3" layer="1"/>
+<contactref element="LED2" pad="C"/>
+<wire x1="84.9125" y1="44.875" x2="82.975" y2="46.8125" width="0.4064" layer="1"/>
+<wire x1="82.975" y1="46.8125" x2="82.125" y2="46.8125" width="0.4064" layer="1"/>
+<via x="82.125" y="46.8125" extent="1-16" drill="0.3"/>
+<wire x1="82.125" y1="46.8125" x2="81.625" y2="46.3125" width="0.4064" layer="15"/>
+<wire x1="81.625" y1="46.3125" x2="81.625" y2="41.6875" width="0.4064" layer="15"/>
+<wire x1="81.625" y1="41.6875" x2="73.4375" y2="33.5" width="0.4064" layer="15"/>
+<wire x1="73.4375" y1="33.5" x2="73.4375" y2="30.625" width="0.4064" layer="15"/>
 </signal>
 <signal name="+5V">
@@
 <wire x1="16.4574" y1="13.0625" x2="14.15" y2="13.0625" width="0.28" layer="1"/>
 <wire x1="14.15" y1="13.0625" x2="14.125" y2="13.0875" width="0.28" layer="1"/>
+<contactref element="LED1" pad="C"/>
+<wire x1="84.975" y1="47.25" x2="84.125" y2="47.25" width="0.4064" layer="1"/>
+<via x="84.125" y="47.25" extent="1-16" drill="0.3"/>
+<wire x1="84.125" y1="47.25" x2="83.1875" y2="46.3125" width="0.4064" layer="15"/>
+<wire x1="83.1875" y1="46.3125" x2="83.1875" y2="30.75" width="0.4064" layer="15"/>
+<wire x1="83.1875" y1="30.75" x2="77.25" y2="24.8125" width="0.4064" layer="15"/>
+<wire x1="77.25" y1="24.8125" x2="75.6875" y2="24.8125" width="0.4064" layer="15"/>
+<wire x1="75.6875" y1="24.8125" x2="74.4375" y2="26.0625" width="0.4064" layer="15"/>
+<wire x1="74.4375" y1="26.0625" x2="74.4375" y2="26.4375" width="0.4064" layer="15"/>
 </signal>
 <signal name="N$2">
@@
 <wire x1="2.35" y1="25.875" x2="2.35" y2="24.875" width="0.6096" layer="16"/>
 <wire x1="2.35" y1="23.875" x2="2.35" y2="24.875" width="0.6096" layer="16"/>
+<contactref element="LED4" pad="C"/>
+<wire x1="84.9125" y1="39.6875" x2="84.9125" y2="39.6625" width="0.4064" layer="1"/>
+<wire x1="84.9125" y1="39.6625" x2="81.5" y2="36.25" width="0.4064" layer="1"/>
+<wire x1="81.5" y1="36.25" x2="81.5" y2="35.75" width="0.4064" layer="1"/>
 </signal>
 <signal name="EDID_SDA">
@@
 <wire x1="67.175" y1="44.625" x2="67.175" y2="47.5125" width="0.8128" layer="16"/>
 <wire x1="67.175" y1="47.5125" x2="66.5625" y2="48.125" width="0.8128" layer="16"/>
+<contactref element="LED3" pad="C"/>
+<wire x1="84.85" y1="42.25" x2="84.1875" y2="42.25" width="0.4064" layer="1"/>
+<wire x1="84.1875" y1="42.25" x2="80.4375" y2="46" width="0.4064" layer="1"/>
+<via x="80.4375" y="46" extent="1-16" drill="0.3"/>
+<wire x1="80.4375" y1="46" x2="79.2125" y2="47.225" width="0.4064" layer="16"/>
+<wire x1="79.2125" y1="47.225" x2="78.625" y2="47.225" width="0.4064" layer="16"/>
 </signal>
 <signal name="N$35">
@@
 <wire x1="3.458" y1="37.124" x2="2.35" y2="36.875" width="0.28" layer="16" curve="25.331246"/>
 </signal>
+<signal name="N$1">
+<contactref element="LED1" pad="A"/>
+<contactref element="R24" pad="2"/>
+<wire x1="86.275" y1="47.25" x2="87.1625" y2="47.25" width="0.4064" layer="1"/>
+</signal>
+<signal name="N$6">
+<contactref element="LED2" pad="A"/>
+<contactref element="R25" pad="2"/>
+<wire x1="86.2125" y1="44.875" x2="87.225" y2="44.875" width="0.4064" layer="1"/>
+</signal>
+<signal name="N$7">
+<contactref element="LED3" pad="A"/>
+<contactref element="R26" pad="2"/>
+<wire x1="86.15" y1="42.25" x2="87.1625" y2="42.25" width="0.4064" layer="1"/>
+</signal>
+<signal name="N$8">
+<contactref element="LED4" pad="A"/>
+<contactref element="R27" pad="2"/>
+<wire x1="86.2125" y1="39.6875" x2="87.1625" y2="39.6875" width="0.4064" layer="1"/>
+</signal>
 </signals>
