File: HDMI_RGB_Bridge/eagle/HDMI_RGB_LVDS/HDMI_RGB_LVDS_fertig_V4.brd (EAGLE design)
At the start: 90 x 60 mm, 87 parts, among them CON1 KLDX-0202-A-LT, CON2 FCI-10029449-111RLF, CON3 XF2M-4015-1A, CON4 FCI-10033526-N3212LF, CON5 MOLEX-53261-0671, CON6 FI-X30SSLA-HF, IC1 WPMDL1300501BD, IC2 WPMDL1300331BD, IC3 TLV1117CDCYR, IC4 AT24C01C-SSHM-B, IC5 TFP401APZP, IC6 ATMEGA48A-AU, IC7 FT232RL, IC8 SN75LVDS83BDGGR, Q1 ATS073ASM-1, T1 IRF9530NSTRRPBF, T2 IRLML2502TRPBF

Commit message: updated schematic and layout
Parts:
- added R28, R29: 10k, SchlegelAr_Master:R0402
Connections:
- net +5V: now also R28.2, R29.2
- net EDID_SCL: now also R29.1
- net EDID_SDA: now also R28.1
Routing:
- net EDID_SCL: track 47.8 -> 50.9 mm
- net +5V: track 74.4 -> 76.2 mm, vias 15 -> 17
- net EDID_SDA: track 49.2 -> 50.6 mm
Changed lines of the file:
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@@
 <layers>
 <layer number="1" name="Top" color="4" fill="1" visible="yes" active="yes"/>
-<layer number="2" name="Route2" color="1" fill="3" visible="yes" active="yes"/>
+<layer number="2" name="Route2" color="1" fill="3" visible="no" active="yes"/>
 <layer number="3" name="Route3" color="4" fill="3" visible="no" active="no"/>
 <layer number="14" name="Route14" color="1" fill="6" visible="no" active="no"/>
@@
 <attribute name="VALUE" x="88.4475" y="41.5925" size="1.27" layer="27" rot="R180"/>
 </element>
+<element name="R28" library="SchlegelAr_Master" package="R0402" value="10k" x="58.5625" y="2.5" rot="MR180"/>
+<element name="R29" library="SchlegelAr_Master" package="R0402" value="10k" x="58.5625" y="1.3125" rot="MR180"/>
 </elements>
 <signals>
@@
 <wire x1="75.6875" y1="24.8125" x2="74.4375" y2="26.0625" width="0.4064" layer="15"/>
 <wire x1="74.4375" y1="26.0625" x2="74.4375" y2="26.4375" width="0.4064" layer="15"/>
+<contactref element="R29" pad="2"/>
+<contactref element="R28" pad="2"/>
+<wire x1="59.2125" y1="2.5" x2="60.0625" y2="2.5" width="0.15" layer="16"/>
+<wire x1="59.2125" y1="1.3125" x2="60.125" y2="1.3125" width="0.15" layer="16"/>
+<via x="60.0625" y="2.5" extent="1-16" drill="0.3"/>
+<via x="60.125" y="1.3125" extent="1-16" drill="0.3"/>
 </signal>
 <signal name="N$2">
@@
 <wire x1="26.625" y1="5.25" x2="36.0625" y2="5.25" width="0.15" layer="16"/>
 <wire x1="36.0625" y1="5.25" x2="38.375" y2="2.9375" width="0.15" layer="16"/>
+<contactref element="R28" pad="1"/>
+<wire x1="57.9125" y1="2.5" x2="57.75" y2="2.5" width="0.15" layer="16"/>
+<wire x1="57.75" y1="2.5" x2="56.875" y2="3.375" width="0.15" layer="16"/>
 </signal>
 <signal name="EDID_SCL">
@@
 <wire x1="26.3125" y1="4.625" x2="36" y2="4.625" width="0.15" layer="16"/>
 <wire x1="36" y1="4.625" x2="38.25" y2="2.375" width="0.15" layer="16"/>
+<contactref element="R29" pad="1"/>
+<wire x1="57.9125" y1="1.3125" x2="56.625" y2="1.3125" width="0.15" layer="16"/>
+<wire x1="56.625" y1="1.3125" x2="55.3125" y2="2.625" width="0.15" layer="16"/>
 </signal>
 <signal name="N$18">
