File: HDMI_RGB_Bridge/eagle/HDMI_RGB_LVDS/HDMI_RGB_LVDS_fertig_V4.sch (EAGLE design)
At the start: 79 parts, among them CON1 KLDX-0202-A-LT, CON2 FCI-10029449-111RLF, CON3 XF2M-4015-1A, CON4 FCI-10033526-N3212LF, CON5 MOLEX-53261-0671, CON6 FI-X30SSLA-HF, IC1 WPMDL1300501BD, IC2 WPMDL1300331BD, IC3 TLV1117CDCYR, IC4 AT24C01C-SSHM-B, IC5 TFP401APZP, IC6 ATMEGA48A-AU, IC7 FT232RL, IC8 SN75LVDS83BDGGR, Q1 ATS073ASM-1, T1 IRF9530NSTRRPBF, T2 IRLML2502TRPBF

Commit message: updated version of V4
Parts:
- added LED1, LED2, LED3, LED4: (no value), SchlegelAr_Master:LED0402
- added R24: 261R, SchlegelAr_Master:R0402
- added R25: 600R, SchlegelAr_Master:R0402
- added R26: 1k5, SchlegelAr_Master:R0402
- added R27: 2k5, SchlegelAr_Master:R0402
- C1: device SchlegelAr_Master:C_POL6X6MM -> SchlegelAr_Master:RSS1C101MCN1GS
- C7, C8: value 10p -> 22p
Connections:
- new net N$1: LED1.A, R24.P$2
- new net N$6: LED2.A, R25.P$2
- new net N$7: LED3.A, R26.P$2
- new net N$8: LED4.A, R27.P$2
- net +12V: now also C1.+, LED4.C; no longer C1.P$1
- net +3V3: now also C2.+, LED2.C; no longer C2.P$1
- net +5V: now also C5.+, LED1.C; no longer C5.P$1
- net +9V6: now also C3.+, LED3.C; no longer C3.P$1
- net GND: now also C1.-, C2.-, C3.-, C5.-, R24.P$1, R25.P$1, R26.P$1, R27.P$1; no longer C1.P$2, C2.P$2, C3.P$2, C5.P$2
Other:
- note added: "26.03.2014"
- note added: "S3: Supply voltage indicator LEDs hinzugefuegt"
Changed lines of the file:
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@@
 <part name="U$5" library="SchlegelAr_Master" deviceset="FRAME_A3_LANDSCAPE" device=""/>
 <part name="CON1" library="SchlegelAr_Master" deviceset="KLDX-0202-A-LT" device=""/>
-<part name="C1" library="SchlegelAr_Master" deviceset="C_POL" device="6X6MM" value="100u"/>
+<part name="C1" library="SchlegelAr_Master" deviceset="RSS1C101MCN1GS" device="" value="100u"/>
 <part name="U$9" library="SchlegelAr_Master" deviceset="GND" device=""/>
 <part name="U$12" library="SchlegelAr_Master" deviceset="GND" device=""/>
@@
 <part name="CON5" library="SchlegelAr_Master" deviceset="MOLEX-53261-0671" device=""/>
 <part name="Q1" library="SchlegelAr_Master" deviceset="ATS073ASM-1" device=""/>
-<part name="C7" library="SchlegelAr_Master" deviceset="C_SMD" device="0402" value="10p"/>
-<part name="C8" library="SchlegelAr_Master" deviceset="C_SMD" device="0402" value="10p"/>
+<part name="C7" library="SchlegelAr_Master" deviceset="C_SMD" device="0402" value="22p"/>
+<part name="C8" library="SchlegelAr_Master" deviceset="C_SMD" device="0402" value="22p"/>
 <part name="C9" library="SchlegelAr_Master" deviceset="C_SMD" device="0402" value="100n"/>
 <part name="U$26" library="SchlegelAr_Master" deviceset="+5V" device=""/>
@@
 <part name="R22" library="SchlegelAr_Master" deviceset="R" device="0402" value="0R"/>
 <part name="R23" library="SchlegelAr_Master" deviceset="R" device="0402" value="0R"/>
+<part name="LED1" library="SchlegelAr_Master" deviceset="LED" device="0402"/>
+<part name="LED2" library="SchlegelAr_Master" deviceset="LED" device="0402"/>
+<part name="LED3" library="SchlegelAr_Master" deviceset="LED" device="0402"/>
+<part name="LED4" library="SchlegelAr_Master" deviceset="LED" device="0402"/>
+<part name="U$70" library="SchlegelAr_Master" deviceset="+5V" device=""/>
+<part name="U$71" library="SchlegelAr_Master" deviceset="+3V3" device=""/>
+<part name="U$72" library="SchlegelAr_Master" deviceset="+9V6" device=""/>
+<part name="U$73" library="SchlegelAr_Master" deviceset="+12V" device=""/>
+<part name="R24" library="SchlegelAr_Master" deviceset="R" device="0402" value="261R"/>
+<part name="R25" library="SchlegelAr_Master" deviceset="R" device="0402" value="600R"/>
+<part name="R26" library="SchlegelAr_Master" deviceset="R" device="0402" value="1k5"/>
+<part name="R27" library="SchlegelAr_Master" deviceset="R" device="0402" value="2k5"/>
+<part name="U$78" library="SchlegelAr_Master" deviceset="GND" device=""/>
+<part name="U$79" library="SchlegelAr_Master" deviceset="GND" device=""/>
+<part name="U$80" library="SchlegelAr_Master" deviceset="GND" device=""/>
+<part name="U$81" library="SchlegelAr_Master" deviceset="GND" device=""/>
 </parts>
 <sheets>
@@
 <text x="10.16" y="172.72" size="2.54" layer="94">25.03.2014</text>
 <text x="35.56" y="172.72" size="2.54" layer="94">S2: Blockschaltbild angepasst, Versorgungsgraph angepasst</text>
+<text x="10.16" y="165.1" size="2.54" layer="94">26.03.2014</text>
+<text x="35.56" y="165.1" size="2.54" layer="94">S3: Supply voltage indicator LEDs hinzugefuegt</text>
 </plain>
 <instances>
@@
 <instance part="U$18" gate="G$1" x="114.3" y="160.02"/>
 <instance part="U$21" gate="G$1" x="78.74" y="119.38"/>
+<instance part="LED1" gate="G$1" x="236.22" y="223.52" rot="R180"/>
+<instance part="LED2" gate="G$1" x="251.46" y="223.52" rot="R180"/>
+<instance part="LED3" gate="G$1" x="266.7" y="223.52" rot="R180"/>
+<instance part="LED4" gate="G$1" x="281.94" y="223.52" rot="R180"/>
+<instance part="U$70" gate="G$1" x="236.22" y="228.6"/>
+<instance part="U$71" gate="G$1" x="251.46" y="228.6"/>
+<instance part="U$72" gate="G$1" x="266.7" y="228.6"/>
+<instance part="U$73" gate="G$1" x="281.94" y="228.6"/>
+<instance part="R24" gate="G$1" x="236.22" y="210.82" rot="R90"/>
+<instance part="R25" gate="G$1" x="251.46" y="210.82" rot="R90"/>
+<instance part="R26" gate="G$1" x="266.7" y="210.82" rot="R90"/>
+<instance part="R27" gate="G$1" x="281.94" y="210.82" rot="R90"/>
+<instance part="U$78" gate="G$1" x="236.22" y="200.66"/>
+<instance part="U$79" gate="G$1" x="251.46" y="200.66"/>
+<instance part="U$80" gate="G$1" x="266.7" y="200.66"/>
+<instance part="U$81" gate="G$1" x="281.94" y="200.66"/>
 </instances>
 <busses>
@@
 <net name="GND" class="0">
 <segment>
-<pinref part="C1" gate="G$1" pin="P$2"/>
+<pinref part="C1" gate="G$1" pin="-"/>
 <pinref part="U$9" gate="G$1" pin="GND"/>
 <wire x1="58.42" y1="175.26" x2="58.42" y2="205.74" width="0.1524" layer="91"/>
@@
 </segment>
 <segment>
-<pinref part="C2" gate="G$1" pin="P$2"/>
+<pinref part="C2" gate="G$1" pin="-"/>
 <wire x1="114.3" y1="175.26" x2="114.3" y2="172.72" width="0.1524" layer="91"/>
 <pinref part="U$13" gate="G$1" pin="GND"/>
@@
 </segment>
 <segment>
-<pinref part="C5" gate="G$1" pin="P$2"/>
+<pinref part="C5" gate="G$1" pin="-"/>
 <pinref part="U$20" gate="G$1" pin="GND"/>
 <wire x1="114.3" y1="205.74" x2="114.3" y2="208.28" width="0.1524" layer="91"/>
@@
 </segment>
 <segment>
-<pinref part="C3" gate="G$1" pin="P$2"/>
+<pinref part="C3" gate="G$1" pin="-"/>
 <wire x1="114.3" y1="132.08" x2="114.3" y2="119.38" width="0.1524" layer="91"/>
 <pinref part="U$11" gate="G$1" pin="GND"/>
@@
 <pinref part="U$21" gate="G$1" pin="GND"/>
 <wire x1="78.74" y1="121.92" x2="78.74" y2="119.38" width="0.1524" layer="91"/>
+</segment>
+<segment>
+<pinref part="R24" gate="G$1" pin="P$1"/>
+<pinref part="U$78" gate="G$1" pin="GND"/>
+<wire x1="236.22" y1="200.66" x2="236.22" y2="205.74" width="0.1524" layer="91"/>
+</segment>
+<segment>
+<pinref part="U$79" gate="G$1" pin="GND"/>
+<pinref part="R25" gate="G$1" pin="P$1"/>
+<wire x1="251.46" y1="205.74" x2="251.46" y2="200.66" width="0.1524" layer="91"/>
+</segment>
+<segment>
+<pinref part="U$80" gate="G$1" pin="GND"/>
+<pinref part="R26" gate="G$1" pin="P$1"/>
+<wire x1="266.7" y1="205.74" x2="266.7" y2="200.66" width="0.1524" layer="91"/>
+</segment>
+<segment>
+<pinref part="U$81" gate="G$1" pin="GND"/>
+<pinref part="R27" gate="G$1" pin="P$1"/>
+<wire x1="281.94" y1="205.74" x2="281.94" y2="200.66" width="0.1524" layer="91"/>
 </segment>
 </net>
@@
 <pinref part="U$14" gate="G$1" pin="+3V3"/>
 <pinref part="IC2" gate="G$1" pin="VOUT"/>
-<pinref part="C2" gate="G$1" pin="P$1"/>
+<pinref part="C2" gate="G$1" pin="+"/>
 <wire x1="114.3" y1="187.96" x2="114.3" y2="182.88" width="0.1524" layer="91"/>
 <junction x="114.3" y="187.96"/>
+</segment>
+<segment>
+<pinref part="U$71" gate="G$1" pin="+3V3"/>
+<pinref part="LED2" gate="G$1" pin="C"/>
+<wire x1="251.46" y1="226.06" x2="251.46" y2="228.6" width="0.1524" layer="91"/>
 </segment>
 </net>
@@
 <wire x1="114.3" y1="220.98" x2="114.3" y2="233.68" width="0.1524" layer="91"/>
 <pinref part="IC1" gate="G$1" pin="VOUT"/>
-<pinref part="C5" gate="G$1" pin="P$1"/>
+<pinref part="C5" gate="G$1" pin="+"/>
 <wire x1="114.3" y1="220.98" x2="114.3" y2="215.9" width="0.1524" layer="91"/>
 <junction x="114.3" y="220.98"/>
+</segment>
+<segment>
+<pinref part="U$70" gate="G$1" pin="+5V"/>
+<pinref part="LED1" gate="G$1" pin="C"/>
+<wire x1="236.22" y1="226.06" x2="236.22" y2="228.6" width="0.1524" layer="91"/>
 </segment>
 </net>
@@
 <junction x="104.14" y="149.86"/>
 <pinref part="U$18" gate="G$1" pin="+9V6"/>
-<pinref part="C3" gate="G$1" pin="P$1"/>
+<pinref part="C3" gate="G$1" pin="+"/>
 <wire x1="114.3" y1="139.7" x2="114.3" y2="149.86" width="0.1524" layer="91"/>
 <junction x="114.3" y="149.86"/>
+</segment>
+<segment>
+<pinref part="U$72" gate="G$1" pin="+9V6"/>
+<pinref part="LED3" gate="G$1" pin="C"/>
+<wire x1="266.7" y1="226.06" x2="266.7" y2="228.6" width="0.1524" layer="91"/>
 </segment>
 </net>
@@
 <wire x1="68.58" y1="220.98" x2="76.2" y2="220.98" width="0.1524" layer="91"/>
 <junction x="68.58" y="220.98"/>
-<pinref part="C1" gate="G$1" pin="P$1"/>
+<pinref part="C1" gate="G$1" pin="+"/>
 <wire x1="58.42" y1="213.36" x2="58.42" y2="220.98" width="0.1524" layer="91"/>
 <junction x="58.42" y="220.98"/>
 <wire x1="68.58" y1="233.68" x2="68.58" y2="220.98" width="0.1524" layer="91"/>
 </segment>
-</net>
+<segment>
+<pinref part="U$73" gate="G$1" pin="+12V"/>
+<pinref part="LED4" gate="G$1" pin="C"/>
+<wire x1="281.94" y1="226.06" x2="281.94" y2="228.6" width="0.1524" layer="91"/>
+</segment>
+</net>
+<net name="N$1" class="0">
+<segment>
+<pinref part="LED1" gate="G$1" pin="A"/>
+<pinref part="R24" gate="G$1" pin="P$2"/>
+<wire x1="236.22" y1="215.9" x2="236.22" y2="218.44" width="0.1524" layer="91"/>
+</segment>
+</net>
+<net name="N$6" class="0">
+<segment>
+<pinref part="LED2" gate="G$1" pin="A"/>
+<pinref part="R25" gate="G$1" pin="P$2"/>
+<wire x1="251.46" y1="215.9" x2="251.46" y2="218.44" width="0.1524" layer="91"/>
+</segment>
+</net>
+<net name="N$7" class="0">
+<segment>
+<pinref part="LED3" gate="G$1" pin="A"/>
+<pinref part="R26" gate="G$1" pin="P$2"/>
+<wire x1="266.7" y1="215.9" x2="266.7" y2="218.44" width="0.1524" layer="91"/>
+</segment>
+</net>
+<net name="N$8" class="0">
+<segment>
+<pinref part="LED4" gate="G$1" pin="A"/>
+<pinref part="R27" gate="G$1" pin="P$2"/>
+<wire x1="281.94" y1="215.9" x2="281.94" y2="218.44" width="0.1524" layer="91"/>
+</segment>
+</net>

Commit message: updated schematic and layout
Parts:
- added R28, R29: 10k, SchlegelAr_Master:R0402
Connections:
- net +5V: now also R28.P$2, R29.P$2
- net EDID_SCL: now also R29.P$1
- net EDID_SDA: now also R28.P$1
Other:
- note added: "29.03.2014"
- note added: "S3: added Pull-Up Resistors on I2C SCL and SDA"
- moved on the sheet: R16
Changed lines of the file:
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@@
 <part name="U$80" library="SchlegelAr_Master" deviceset="GND" device=""/>
 <part name="U$81" library="SchlegelAr_Master" deviceset="GND" device=""/>
+<part name="R28" library="SchlegelAr_Master" deviceset="R" device="0402" value="10k"/>
+<part name="R29" library="SchlegelAr_Master" deviceset="R" device="0402" value="10k"/>
+<part name="U$82" library="SchlegelAr_Master" deviceset="+5V" device=""/>
+<part name="U$84" library="SchlegelAr_Master" deviceset="+5V" device=""/>
 </parts>
 <sheets>
@@
 <text x="10.16" y="165.1" size="2.54" layer="94">26.03.2014</text>
 <text x="35.56" y="165.1" size="2.54" layer="94">S3: Supply voltage indicator LEDs hinzugefuegt</text>
+<text x="10.16" y="157.48" size="2.54" layer="94">29.03.2014</text>
+<text x="35.56" y="157.48" size="2.54" layer="94">S3: added Pull-Up Resistors on I2C SCL and SDA</text>
 </plain>
 <instances>
@@
 <instance part="C8" gate="G$1" x="149.86" y="210.82"/>
 <instance part="C9" gate="G$1" x="160.02" y="157.48" rot="R270"/>
-<instance part="U$26" gate="G$1" x="167.64" y="236.22"/>
+<instance part="U$26" gate="G$1" x="182.88" y="246.38"/>
 <instance part="U$27" gate="G$1" x="144.78" y="106.68"/>
 <instance part="JP5" gate="G$1" x="139.7" y="114.3" rot="R90"/>
@@
 <instance part="U$46" gate="G$1" x="17.78" y="149.86"/>
 <instance part="U$48" gate="G$1" x="160.02" y="149.86"/>
-<instance part="R16" gate="G$1" x="175.26" y="233.68"/>
+<instance part="R16" gate="G$1" x="182.88" y="238.76" rot="R270"/>
 <instance part="U$49" gate="G$1" x="322.58" y="215.9" rot="R90"/>
 <instance part="R17" gate="G$1" x="144.78" y="127" rot="R90"/>
@@
 <instance part="R22" gate="G$1" x="76.2" y="190.5"/>
 <instance part="R23" gate="G$1" x="86.36" y="187.96"/>
+<instance part="R28" gate="G$1" x="160.02" y="228.6" rot="R90"/>
+<instance part="R29" gate="G$1" x="167.64" y="228.6" rot="R90"/>
+<instance part="U$82" gate="G$1" x="167.64" y="246.38"/>
+<instance part="U$84" gate="G$1" x="160.02" y="246.38"/>
 </instances>
 <busses>
@@
 <segment>
 <pinref part="R16" gate="G$1" pin="P$2"/>
-<wire x1="182.88" y1="233.68" x2="182.88" y2="223.52" width="0.1524" layer="91"/>
+<wire x1="182.88" y1="231.14" x2="182.88" y2="223.52" width="0.1524" layer="91"/>
 <wire x1="182.88" y1="223.52" x2="185.42" y2="223.52" width="0.1524" layer="91"/>
-<wire x1="180.34" y1="233.68" x2="182.88" y2="233.68" width="0.1524" layer="91"/>
-<wire x1="182.88" y1="233.68" x2="185.42" y2="233.68" width="0.1524" layer="91"/>
-<label x="185.42" y="233.68" size="1.27" layer="95" xref="yes"/>
-<junction x="182.88" y="233.68"/>
+<wire x1="182.88" y1="233.68" x2="182.88" y2="231.14" width="0.1524" layer="91"/>
+<wire x1="182.88" y1="231.14" x2="185.42" y2="231.14" width="0.1524" layer="91"/>
+<label x="185.42" y="231.14" size="1.27" layer="95" xref="yes"/>
+<junction x="182.88" y="231.14"/>
 <pinref part="IC6" gate="G$1" pin="PC6(PCINT14/RESET)"/>
 </segment>
@@
 <segment>
 <pinref part="U$26" gate="G$1" pin="+5V"/>
-<wire x1="167.64" y1="236.22" x2="167.64" y2="233.68" width="0.1524" layer="91"/>
-<wire x1="167.64" y1="233.68" x2="170.18" y2="233.68" width="0.1524" layer="91"/>
+<wire x1="182.88" y1="246.38" x2="182.88" y2="243.84" width="0.1524" layer="91"/>
 <pinref part="R16" gate="G$1" pin="P$1"/>
 </segment>
@@
 <pinref part="U$35" gate="G$1" pin="+5V"/>
 </segment>
+<segment>
+<pinref part="R29" gate="G$1" pin="P$2"/>
+<pinref part="U$82" gate="G$1" pin="+5V"/>
+<wire x1="167.64" y1="246.38" x2="167.64" y2="233.68" width="0.1524" layer="91"/>
+</segment>
+<segment>
+<pinref part="R28" gate="G$1" pin="P$2"/>
+<pinref part="U$84" gate="G$1" pin="+5V"/>
+<wire x1="160.02" y1="246.38" x2="160.02" y2="233.68" width="0.1524" layer="91"/>
+</segment>
 </net>
 <net name="EDID_SDA" class="0">
 <segment>
-<wire x1="185.42" y1="218.44" x2="182.88" y2="218.44" width="0.1524" layer="91"/>
-<label x="182.88" y="218.44" size="1.27" layer="95" rot="R180" xref="yes"/>
+<wire x1="185.42" y1="218.44" x2="160.02" y2="218.44" width="0.1524" layer="91"/>
+<label x="157.48" y="218.44" size="1.27" layer="95" rot="R180" xref="yes"/>
 <pinref part="IC6" gate="G$1" pin="PC4(SDA/ADC4/PCINT12)"/>
+<pinref part="R28" gate="G$1" pin="P$1"/>
+<wire x1="160.02" y1="218.44" x2="157.48" y2="218.44" width="0.1524" layer="91"/>
+<wire x1="160.02" y1="223.52" x2="160.02" y2="218.44" width="0.1524" layer="91"/>
+<junction x="160.02" y="218.44"/>
 </segment>
 <segment>
@@
 <net name="EDID_SCL" class="0">
 <segment>
-<wire x1="185.42" y1="220.98" x2="182.88" y2="220.98" width="0.1524" layer="91"/>
-<label x="182.88" y="220.98" size="1.27" layer="95" rot="R180" xref="yes"/>
+<wire x1="185.42" y1="220.98" x2="167.64" y2="220.98" width="0.1524" layer="91"/>
+<label x="157.48" y="220.98" size="1.27" layer="95" rot="R180" xref="yes"/>
 <pinref part="IC6" gate="G$1" pin="PC5(SCL/ADC5/PCINT13)"/>
-</segment>
-<segment>
+<pinref part="R29" gate="G$1" pin="P$1"/>
+<wire x1="167.64" y1="220.98" x2="157.48" y2="220.98" width="0.1524" layer="91"/>
+<wire x1="167.64" y1="223.52" x2="167.64" y2="220.98" width="0.1524" layer="91"/>
+<junction x="167.64" y="220.98"/>
+</segment>
+<segment>

Commit message: end of workday 01.04.2014
Other:
- note added: "ATmega88"
- note added: "Atmel ATmega88"
- note removed: "ATmega48"
- note removed: "Atmel ATmega32U4"
Changed lines of the file:
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@@
 <text x="22.86" y="175.26" size="2.54" layer="94">I2C EEPROM
 Atmel AT2401C</text>
-<text x="22.86" y="144.78" size="2.54" layer="94">Atmel ATmega32U4</text>
+<text x="22.86" y="144.78" size="2.54" layer="94">Atmel ATmega88</text>
 <text x="40.64" y="195.58" size="2.54" layer="97">Edid data</text>
 <text x="134.62" y="223.52" size="2.54" layer="97">RGB Bus</text>
@@
 <rectangle x1="182.88" y1="114.3" x2="360.68" y2="116.84" layer="94"/>
 <text x="182.88" y="116.84" size="3.81" layer="94">+5V</text>
-<text x="185.42" y="99.06" size="3.81" layer="92">ATmega48</text>
+<text x="185.42" y="99.06" size="3.81" layer="92">ATmega88</text>
 <text x="233.68" y="99.06" size="3.81" layer="92">I2C EEPROM</text>
 <text x="281.94" y="99.06" size="3.81" layer="92">FT232RL</text>
