File: HDMI_RGB_Bridge/eagle/HDMI_RGB_LVDS/HDMI_RGB_LVDS_fertig_V5.sch (EAGLE design)
At the start: 79 parts, among them CON1 KLDX-0202-A-LT, CON2 FCI-10029449-111RLF, CON3 XF2M-4015-1A, CON4 FCI-10033526-N3212LF, CON5 MOLEX-53261-0671, CON6 FI-X30SSLA-HF, IC1 WPMDL1300501BD, IC2 WPMDL1300331BD, IC3 TLV1117CDCYR, IC4 AT24C01C-SSHM-B, IC5 TFP401APZP, IC6 ATMEGA48A-AU, IC7 FT232RL, IC8 SN75LVDS83BDGGR, Q1 ATS073ASM-1, T1 IRF9530NSTRRPBF, T2 IRLML2502TRPBF

Commit message: end of workday 01.04.2014
Parts:
- removed D1: BZG03C15TR3, SchlegelAr_Master:BZG03C15TR3
- removed IC1: WPMDL1300501BD, SchlegelAr_Master:WPMDL1300501BD
- removed IC3: TLV1117CDCYR, SchlegelAr_Master:TLV1117CDCYR
- removed R14: 31k4, SchlegelAr_Master:R0402
- removed R21: 140R, SchlegelAr_Master:R2512
- added C25, C26, C27, C28, C29, C30, C31, C32, C33: 100n, SchlegelAr_Master:C_SMD0402
- added C34, C35, C36: 10u, SchlegelAr_Master:C_POL4X4MM
- added LED2, LED4: (no value), SchlegelAr_Master:LED0402
- added R25: 600R, SchlegelAr_Master:R0402
- added R27: 2k5, SchlegelAr_Master:R0402
- added R28, R29: 10k, SchlegelAr_Master:R0402
- C3: value 10u -> 100n; device SchlegelAr_Master:C_POL4X4MM -> SchlegelAr_Master:C_SMD0402
- R13: value 4k7 -> 10k
- R20: value 140R -> 15R
- R7: value 100R -> 10k
Connections:
- removed net +9V6: C3.+, IC3.OUT, IC3.OUT1, R13.P$2, R20.P$2, R21.P$2
- removed net N$35: IC3.GND, R13.P$1, R14.P$1
- new net +5V_USB: C12.P$1, CON4.VBUS, IC7.!RESET, IC7.VCC, IC7.VCCIO, R13.P$2
- new net N$6: LED2.A, R25.P$2
- new net N$8: LED4.A, R27.P$2
- net +12V: now also C34.+, LED4.C, R20.P$2; no longer D1.C, IC1.VIN, IC3.IN
- net +3V3: now also C25.P$2, C26.P$2, C27.P$2, C28.P$2, C29.P$2, C3.P$2, C30.P$2, C31.P$2, C32.P$2, C33.P$2, C35.+, C36.+, LED2.C
- net +5V: now also R13.P$1, R28.P$2, R29.P$2; no longer C12.P$1, C5.+, CON4.VBUS, IC1.VOUT, IC7.!RESET, IC7.VCC, IC7.VCCIO
- net EDID_SCL: now also R29.P$1
- net EDID_SDA: now also R28.P$1
- net GND: now also C25.P$1, C26.P$1, C27.P$1, C28.P$1, C29.P$1, C3.P$1, C30.P$1, C31.P$1, C32.P$1, C33.P$1, C34.-, C35.-, C36.-, R25.P$1, R27.P$1; no longer C3.-, C5.-, IC1.GND, IC1.PGND, R14.P$2
- net N$4: no longer D1.A
- net N$57: no longer R21.P$1
Other:
- note added: "26.03.2014"
- note added: "29.03.2014"
- note added: "ATmega88"
- note added: "Atmel ATmega88"
- note added: "NOTE: LCD Backlight 9.6V@180mA R = (12V-9.6V)/180mA = 15 Ohm"
- note added: "NOTE: Max. Input 12V"
- note added: "S3: Supply voltage indicator LEDs hinzugefuegt"
- note added: "S3: added Pull-Up Resistors on I2C SCL and SDA"
- note removed: "ATmega48"
- note removed: "Atmel ATmega32U4"
- note removed: "NOTE: LCD Backlight 9.6V@170mA => R = 70 Ohm, 2W"
- note removed: "NOTE: WPMDL1300501BD has internal pullup on EN-pin."
- moved on the sheet: C13, C14, C2, C4, C5, C6, IC2, R1, R16

Commit message: schematic and layout adapted
Parts:
- removed C5: 10u, SchlegelAr_Master:C_POL4X4MM
- removed LED4: (no value), SchlegelAr_Master:LED0402
- added LED1: (no value), SchlegelAr_Master:LED0402
- added R14: 22R, SchlegelAr_Master:R0402
- C16, C18, C20: value 0.1u -> 100n
- IC6: value ATMEGA48A-AU -> ATMEGA88PA
- R19: value 10k -> 5k
- T1: value IRF9530NSTRRPBF -> IRLML5203TRPBF; device SchlegelAr_Master:IRF9530NSTRRPBF -> SchlegelAr_Master:IRLML5203TRPBF
Connections:
- new net N$1: IC6.PB1(OC1A/PCINT1), R14.P$1
- net +12V: now also LED2.C; no longer LED4.C
- net +3V3: now also LED1.C; no longer LED2.C
- net AVR_PWM: now also R14.P$2; no longer IC6.PB1(OC1A/PCINT1)
- net N$6: now also LED1.A; no longer LED2.A
- net N$8: now also LED2.A; no longer LED4.A
Other:
- note added: "I2C EEPROM Atmel AT24C01"
- note added: "NOTE: LCD Backlight 9.6V@180mA R20 = (12V-9.6V)/180mA = 15 Ohm"
- note added: "RGB Display TY700TFT800480"
- note removed: "+9.6V"
- note removed: "I2C EEPROM Atmel AT2401C"
- note removed: "NOTE: LCD Backlight 9.6V@180mA R = (12V-9.6V)/180mA = 15 Ohm"
- note removed: "NOTE: VCCIO is +5V because AVR is +5V"
- note removed: "RGB Display"
- moved on the sheet: C13, C14, C15, C16, C17, C18, C19, C2, C20, C21, C22, C25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
