File: Teil_A/hardware/Gnublin_Extended_8080/gnublin_ext_8080.brd (EAGLE design)
At the start: 134.5 x 84 mm, 7 parts

Commit message: end of workday 29.07.2014
Connections:
- net +3V3: now also R2.2
- net GND: no longer R2.2
Routing:
- net +3V3: track 32.6 -> 37.2 mm, vias 4 -> 5
- net GND: track 26.1 -> 24.6 mm
Changed lines of the file:
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@@
 <via x="114.3" y="6.2" extent="1-16" drill="0.6" diameter="1.6764"/>
 <via x="16" y="13.7" extent="1-16" drill="0.6" diameter="1.6764"/>
-<contactref element="R2" pad="2"/>
-<wire x1="79.35" y1="17.5" x2="77.9" y2="17.5" width="0.4" layer="16"/>
 </signal>
 <signal name="+3V3">
@@
 <contactref element="JP3" pad="2"/>
 <contactref element="R1" pad="2"/>
+<contactref element="R2" pad="2"/>
 <contactref element="C1" pad="1"/>
 <contactref element="R3" pad="2"/>
@@
 <wire x1="66.9" y1="64.8" x2="67.2" y2="65.1" width="0.4" layer="16"/>
 <wire x1="67.2" y1="65.1" x2="67.75" y2="65.65" width="0.4" layer="16"/>
+<wire x1="79.35" y1="17.5" x2="77.9" y2="17.5" width="0.4" layer="16"/>
+<wire x1="77.9" y1="17.5" x2="76.7" y2="18.7" width="0.4" layer="16"/>
+<via x="76.7" y="18.7" extent="1-16" drill="0.6" diameter="1.6764"/>
+<wire x1="76.7" y1="18.7" x2="76.1" y2="18.7" width="0.4" layer="1"/>
+<wire x1="76.1" y1="18.7" x2="75.5" y2="19.3" width="0.4" layer="1"/>
 <wire x1="84.75" y1="17.5" x2="84.75" y2="18.05" width="0.4" layer="16"/>
 <wire x1="84.75" y1="18.05" x2="85.8" y2="19.1" width="0.4" layer="16"/>
