File: Teil_B/HDMI_RGB_Bridge/eagle/HDMI_RGB_LVDS/HDMI_RGB_LVDS_V10.sch (EAGLE design)
At the start: 95 parts, among them CON1 KLDX-0202-A-LT, CON2 FCI-10029449-111RLF, CON3 XF2M-4015-1A, CON4 FCI-10033526-N3212LF, CON5 MOLEX-53261-0671, CON6 FI-X30SSLA-HF, IC2 WPMDL1300331BD, IC4 AT24C01C-SSHM-B, IC5 TFP401APZP, IC6 ATMEGA88PA, IC7 FT232RL, IC8 SN75LVDS83BDGGR, Q1 ATS073ASM-1, T1 IRLML5203TRPBF, T2 IRLML2502TRPBF

Commit message: end of workday 13.08.2014
Other:
- note added: "NOTE: Input 12V"
- note added: "Pixelselect: The DVI RX output is configurable with pin "PIXS". When PIXS is Low, RGB data is output on 24 bits (QE[23:0]). When PIXS is High, RGB data is split odd/even on 48-bits. Jumper present: 24 BIT No Jumper: 48 Bit"
- note removed: "NOTE: Max. Input 12V"
- note removed: "Pixelselect: Selects between one or two pixels per clock output modes. During the 2-pixel/clck mode, both even pixels and odd pixels, are output in tandem on a given clock cycle. During the 1-pixel/clock mode, even and odd pixels are output sequentially, on the same time, with the even pixel first, on the even pixel bus. Jumper present: 1-pixel/clock No Jumper: 2-pixel/clock"
- moved on the sheet: LED1, LED2, R25, R27
